File: thpd-kb01.kicad_pcb (KiCad board)
At the start: 4 copper layers, 344 parts, among them J1 USB_C_Receptacle_USB2.0, SW1 SW_Push, SW2 SW_SPDT, SW3 Rotary_Encoder_Switch, U1 XC6206PxxxMR, U2 USBLC6-2SC6, U3 NHD-C12832A1Z, U4 STM32F072C8Tx

Commit message: WIP
Parts:
- F1: footprint Fuse:Fuse_1206_3216Metric -> Fuse:Fuse_0603_1608Metric
- moved R10 8.91 mm to (285.6, 119.0)
- moved D102 8.21 mm to (394.0, 88.9), turned to 0 degrees
- moved J1 5.85 mm to (327.6, 85.2)
- moved R1 3.41 mm to (326.0, 92.8)
- moved C21 2.26 mm to (385.9, 85.6)
- moved C20 1.48 mm to (385.9, 97.8)
- moved R2 1.42 mm to (329.6, 92.9)
- moved C2 1.32 mm to (321.6, 97.2)
- moved C13 1.21 mm to (365.6, 98.0)
- moved C1 1.20 mm to (327.8, 99.6)
- moved C14 1.19 mm to (367.9, 97.6)
- moved C12 1.16 mm to (362.7, 98.0)
- moved C19 1.09 mm to (359.8, 97.9)
- moved C15 0.86 mm to (369.4, 97.6)
- moved C16 0.83 mm to (370.9, 97.6)
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Connections:
- D1 pad 1: /keys_matrix/ROW0 -> ROW0
- D10 pad 1: /keys_matrix/ROW0 -> ROW0
- D100 pad 1: /keys_matrix/ROW5 -> ROW5
- D101 pad 1: /keys_matrix/ROW5 -> ROW5
- D102 pad 1: /keys_matrix/ROW0 -> ROW0
- D11 pad 1: /keys_matrix/ROW0 -> ROW0
- D12 pad 1: /keys_matrix/ROW0 -> ROW0
- D13 pad 1: /keys_matrix/ROW0 -> ROW0
- D14 pad 1: /keys_matrix/ROW0 -> ROW0
- D15 pad 1: /keys_matrix/ROW0 -> ROW0
- D16 pad 1: /keys_matrix/ROW0 -> ROW0
- D17 pad 1: /keys_matrix/ROW1 -> ROW1
- D18 pad 1: /keys_matrix/ROW1 -> ROW1
- D19 pad 1: /keys_matrix/ROW1 -> ROW1
- D2 pad 1: /keys_matrix/ROW0 -> ROW0
- D20 pad 1: /keys_matrix/ROW1 -> ROW1
- D21 pad 1: /keys_matrix/ROW1 -> ROW1
- D22 pad 1: /keys_matrix/ROW1 -> ROW1
- D23 pad 1: /keys_matrix/ROW1 -> ROW1
- D24 pad 1: /keys_matrix/ROW1 -> ROW1
- D25 pad 1: /keys_matrix/ROW1 -> ROW1
- D26 pad 1: /keys_matrix/ROW1 -> ROW1
- D27 pad 1: /keys_matrix/ROW1 -> ROW1
- D28 pad 1: /keys_matrix/ROW1 -> ROW1
- D29 pad 1: /keys_matrix/ROW1 -> ROW1
- D3 pad 1: /keys_matrix/ROW0 -> ROW0
- D30 pad 1: /keys_matrix/ROW1 -> ROW1
- D31 pad 1: /keys_matrix/ROW1 -> ROW1
- D32 pad 1: /keys_matrix/ROW1 -> ROW1
- D33 pad 1: /keys_matrix/ROW1 -> ROW1
- D34 pad 1: /keys_matrix/ROW1 -> ROW1
- D35 pad 1: /keys_matrix/ROW1 -> ROW1
- D36 pad 1: /keys_matrix/ROW2 -> ROW2
- D37 pad 1: /keys_matrix/ROW2 -> ROW2
- D38 pad 1: /keys_matrix/ROW2 -> ROW2
- D39 pad 1: /keys_matrix/ROW2 -> ROW2
- D4 pad 1: /keys_matrix/ROW0 -> ROW0
- D40 pad 1: /keys_matrix/ROW2 -> ROW2
- D41 pad 1: /keys_matrix/ROW2 -> ROW2
- D42 pad 1: /keys_matrix/ROW2 -> ROW2
- D43 pad 1: /keys_matrix/ROW2 -> ROW2
- D44 pad 1: /keys_matrix/ROW2 -> ROW2
- D45 pad 1: /keys_matrix/ROW2 -> ROW2
- D46 pad 1: /keys_matrix/ROW2 -> ROW2
- D47 pad 1: /keys_matrix/ROW2 -> ROW2
- D48 pad 1: /keys_matrix/ROW2 -> ROW2
- D49 pad 1: /keys_matrix/ROW2 -> ROW2
- D5 pad 1: /keys_matrix/ROW0 -> ROW0
- D50 pad 1: /keys_matrix/ROW2 -> ROW2
- D51 pad 1: /keys_matrix/ROW2 -> ROW2
- D52 pad 1: /keys_matrix/ROW2 -> ROW2
- D53 pad 1: /keys_matrix/ROW2 -> ROW2
- D54 pad 1: /keys_matrix/ROW2 -> ROW2
- D55 pad 1: /keys_matrix/ROW3 -> ROW3
- D56 pad 1: /keys_matrix/ROW3 -> ROW3
- D57 pad 1: /keys_matrix/ROW3 -> ROW3
- D58 pad 1: /keys_matrix/ROW3 -> ROW3
- D59 pad 1: /keys_matrix/ROW3 -> ROW3
- D6 pad 1: /keys_matrix/ROW0 -> ROW0
- D60 pad 1: /keys_matrix/ROW3 -> ROW3
- D61 pad 1: /keys_matrix/ROW3 -> ROW3
- D62 pad 1: /keys_matrix/ROW3 -> ROW3
- D63 pad 1: /keys_matrix/ROW3 -> ROW3
- D64 pad 1: /keys_matrix/ROW3 -> ROW3
- D65 pad 1: /keys_matrix/ROW3 -> ROW3
- D66 pad 1: /keys_matrix/ROW3 -> ROW3
- D67 pad 1: /keys_matrix/ROW3 -> ROW3
- D68 pad 1: /keys_matrix/ROW3 -> ROW3
- D69 pad 1: /keys_matrix/ROW3 -> ROW3
- D7 pad 1: /keys_matrix/ROW0 -> ROW0
- D70 pad 1: /keys_matrix/ROW3 -> ROW3
- D71 pad 1: /keys_matrix/ROW3 -> ROW3
- D72 pad 1: /keys_matrix/ROW4 -> ROW4
- D73 pad 1: /keys_matrix/ROW4 -> ROW4
- D74 pad 1: /keys_matrix/ROW4 -> ROW4
- D75 pad 1: /keys_matrix/ROW4 -> ROW4
- D76 pad 1: /keys_matrix/ROW4 -> ROW4
- D77 pad 1: /keys_matrix/ROW4 -> ROW4
- D78 pad 1: /keys_matrix/ROW4 -> ROW4
- D79 pad 1: /keys_matrix/ROW4 -> ROW4
- D8 pad 1: /keys_matrix/ROW0 -> ROW0
- D80 pad 1: /keys_matrix/ROW4 -> ROW4
- D81 pad 1: /keys_matrix/ROW4 -> ROW4
- D82 pad 1: /keys_matrix/ROW4 -> ROW4
- D83 pad 1: /keys_matrix/ROW4 -> ROW4
- D84 pad 1: /keys_matrix/ROW4 -> ROW4
- D85 pad 1: /keys_matrix/ROW4 -> ROW4
- D86 pad 1: /keys_matrix/ROW4 -> ROW4
- D87 pad 1: /keys_matrix/ROW4 -> ROW4
- D88 pad 1: /keys_matrix/ROW4 -> ROW4
- D89 pad 1: /keys_matrix/ROW4 -> ROW4
- D9 pad 1: /keys_matrix/ROW0 -> ROW0
- D90 pad 1: /keys_matrix/ROW5 -> ROW5
- D91 pad 1: /keys_matrix/ROW5 -> ROW5
- D92 pad 1: /keys_matrix/ROW5 -> ROW5
- D93 pad 1: /keys_matrix/ROW5 -> ROW5
- D94 pad 1: /keys_matrix/ROW5 -> ROW5
- D95 pad 1: /keys_matrix/ROW5 -> ROW5
- D96 pad 1: /keys_matrix/ROW5 -> ROW5
- D97 pad 1: /keys_matrix/ROW5 -> ROW5
- D98 pad 1: /keys_matrix/ROW5 -> ROW5
- D99 pad 1: /keys_matrix/ROW5 -> ROW5
- MX1 pad 1: /keys_matrix/COL0 -> COL0
- MX10 pad 1: /keys_matrix/COL9 -> COL9
- MX100 pad 1: /keys_matrix/COL15 -> COL15
- MX101 pad 1: /keys_matrix/COL17 -> COL17
- MX11 pad 1: /keys_matrix/COL10 -> COL10
- MX12 pad 1: /keys_matrix/COL11 -> COL11
- MX13 pad 1: /keys_matrix/COL12 -> COL12
- MX14 pad 1: /keys_matrix/COL13 -> COL13
- MX15 pad 1: /keys_matrix/COL14 -> COL14
- MX16 pad 1: /keys_matrix/COL15 -> COL15
- MX17 pad 1: /keys_matrix/COL0 -> COL0
- MX18 pad 1: /keys_matrix/COL1 -> COL1
- MX19 pad 1: /keys_matrix/COL2 -> COL2
- MX2 pad 1: /keys_matrix/COL1 -> COL1
- MX20 pad 1: /keys_matrix/COL3 -> COL3
- MX21 pad 1: /keys_matrix/COL4 -> COL4
- MX22 pad 1: /keys_matrix/COL5 -> COL5
- MX23 pad 1: /keys_matrix/COL6 -> COL6
- MX24 pad 1: /keys_matrix/COL7 -> COL7
- MX25 pad 1: /keys_matrix/COL8 -> COL8
- MX26 pad 1: /keys_matrix/COL9 -> COL9
- MX27 pad 1: /keys_matrix/COL10 -> COL10
- MX28 pad 1: /keys_matrix/COL11 -> COL11
- MX29 pad 1: /keys_matrix/COL12 -> COL12
- MX3 pad 1: /keys_matrix/COL2 -> COL2
- MX30 pad 1: /keys_matrix/COL13 -> COL13
- MX31 pad 1: /keys_matrix/COL14 -> COL14
- MX32 pad 1: /keys_matrix/COL15 -> COL15
- MX33 pad 1: /keys_matrix/COL16 -> COL16
- MX34 pad 1: /keys_matrix/COL17 -> COL17
- MX35 pad 1: ROT_SW_COL -> COL18
- MX36 pad 1: /keys_matrix/COL0 -> COL0
- MX37 pad 1: /keys_matrix/COL1 -> COL1
- MX38 pad 1: /keys_matrix/COL2 -> COL2
- MX39 pad 1: /keys_matrix/COL3 -> COL3
- MX4 pad 1: /keys_matrix/COL3 -> COL3
- MX40 pad 1: /keys_matrix/COL4 -> COL4
- MX41 pad 1: /keys_matrix/COL5 -> COL5
- MX42 pad 1: /keys_matrix/COL6 -> COL6
- MX43 pad 1: /keys_matrix/COL7 -> COL7
- MX44 pad 1: /keys_matrix/COL8 -> COL8
- MX45 pad 1: /keys_matrix/COL9 -> COL9
- MX46 pad 1: /keys_matrix/COL10 -> COL10
- MX47 pad 1: /keys_matrix/COL11 -> COL11
- MX48 pad 1: /keys_matrix/COL12 -> COL12
- MX49 pad 1: /keys_matrix/COL13 -> COL13
- MX5 pad 1: /keys_matrix/COL4 -> COL4
- MX50 pad 1: /keys_matrix/COL14 -> COL14
- MX51 pad 1: /keys_matrix/COL15 -> COL15
- MX52 pad 1: /keys_matrix/COL16 -> COL16
- MX53 pad 1: /keys_matrix/COL17 -> COL17
- MX54 pad 1: ROT_SW_COL -> COL18
- MX55 pad 1: /keys_matrix/COL0 -> COL0
- MX56 pad 1: /keys_matrix/COL1 -> COL1
- MX57 pad 1: /keys_matrix/COL2 -> COL2
- MX58 pad 1: /keys_matrix/COL3 -> COL3
- MX59 pad 1: /keys_matrix/COL4 -> COL4
- MX6 pad 1: /keys_matrix/COL5 -> COL5
- MX60 pad 1: /keys_matrix/COL5 -> COL5
- MX61 pad 1: /keys_matrix/COL6 -> COL6
- MX62 pad 1: /keys_matrix/COL7 -> COL7
- MX63 pad 1: /keys_matrix/COL8 -> COL8
- MX64 pad 1: /keys_matrix/COL9 -> COL9
- MX65 pad 1: /keys_matrix/COL10 -> COL10
- MX66 pad 1: /keys_matrix/COL11 -> COL11
- MX67 pad 1: /keys_matrix/COL12 -> COL12
- MX68 pad 1: /keys_matrix/COL14 -> COL14
- MX69 pad 1: /keys_matrix/COL15 -> COL15
- MX7 pad 1: /keys_matrix/COL6 -> COL6
- MX70 pad 1: /keys_matrix/COL16 -> COL16
- MX71 pad 1: /keys_matrix/COL17 -> COL17
- MX72 pad 1: /keys_matrix/COL0 -> COL0
- MX73 pad 1: /keys_matrix/COL1 -> COL1
- MX74 pad 1: /keys_matrix/COL2 -> COL2
- MX75 pad 1: /keys_matrix/COL3 -> COL3
- MX76 pad 1: /keys_matrix/COL4 -> COL4
- MX77 pad 1: /keys_matrix/COL5 -> COL5
- MX78 pad 1: /keys_matrix/COL6 -> COL6
- MX79 pad 1: /keys_matrix/COL7 -> COL7
- MX8 pad 1: /keys_matrix/COL7 -> COL7
- MX80 pad 1: /keys_matrix/COL8 -> COL8
- MX81 pad 1: /keys_matrix/COL9 -> COL9
- MX82 pad 1: /keys_matrix/COL10 -> COL10
- MX83 pad 1: /keys_matrix/COL12 -> COL12
- MX84 pad 1: /keys_matrix/COL13 -> COL13
- MX85 pad 1: /keys_matrix/COL14 -> COL14
- MX86 pad 1: /keys_matrix/COL15 -> COL15
- MX87 pad 1: /keys_matrix/COL16 -> COL16
- MX88 pad 1: /keys_matrix/COL17 -> COL17
- MX89 pad 1: ROT_SW_COL -> COL18
- MX9 pad 1: /keys_matrix/COL8 -> COL8
- MX90 pad 1: /keys_matrix/COL0 -> COL0
- MX91 pad 1: /keys_matrix/COL1 -> COL1
- MX92 pad 1: /keys_matrix/COL2 -> COL2
- MX93 pad 1: /keys_matrix/COL5 -> COL5
- MX94 pad 1: /keys_matrix/COL9 -> COL9
- MX95 pad 1: /keys_matrix/COL10 -> COL10
- MX96 pad 1: /keys_matrix/COL11 -> COL11
- MX97 pad 1: /keys_matrix/COL12 -> COL12
- MX98 pad 1: /keys_matrix/COL13 -> COL13
- MX99 pad 1: /keys_matrix/COL14 -> COL14
- R10 pad 2: (no net) -> /led_matrix/DIN
- SW3 pad S1: ROT_SW_COL -> COL18
- U4 pad 11: (no net) -> ROW5
- U4 pad 12: (no net) -> /led_matrix/DIN
- U4 pad 18: (no net) -> COL9
- U4 pad 19: (no net) -> COL10
- U4 pad 2: (no net) -> ROW0
- U4 pad 20: (no net) -> COL11
- U4 pad 21: (no net) -> COL12
- U4 pad 22: (no net) -> COL13
- U4 pad 25: (no net) -> ROT_A
- U4 pad 26: (no net) -> ROT_B
- U4 pad 27: (no net) -> COL14
- U4 pad 28: (no net) -> COL15
- U4 pad 29: (no net) -> COL16
- U4 pad 3: (no net) -> ROW1
- U4 pad 30: (no net) -> COL17
- U4 pad 31: (no net) -> COL18
- U4 pad 37: (no net) -> COL0
- U4 pad 38: (no net) -> COL1
- U4 pad 39: (no net) -> COL2
- U4 pad 4: (no net) -> ROW2
- U4 pad 40: (no net) -> COL3
- U4 pad 41: (no net) -> COL4
- U4 pad 42: (no net) -> COL5
- U4 pad 43: (no net) -> COL6
- U4 pad 45: (no net) -> COL7
- U4 pad 46: (no net) -> COL8
- U4 pad 5: (no net) -> ROW3
- U4 pad 6: (no net) -> ROW4
Other:
- board outline added: 388 x 116 mm

Commit message: WIP
Parts:
- moved C1 11.3 mm to (339.0, 98.3)
- moved C2 11.3 mm to (332.8, 95.9)
- moved U1 11.3 mm to (335.4, 95.9)
- moved F1 9.83 mm to (338.9, 93.5), turned to 90 degrees
- moved R3 8.42 mm to (326.3, 99.2)
- moved R4 8.42 mm to (328.4, 99.2)
- moved U2 8.39 mm to (327.4, 96.0)
- moved C8 1.61 mm to (287.7, 121.6)
- moved C9 1.61 mm to (300.9, 125.6)
- moved R10 1.61 mm to (284.2, 119.8)
- moved U4 1.61 mm to (295.0, 122.6)
- moved C10 1.61 mm to (302.1, 125.6)
- moved C3 1.61 mm to (298.0, 115.7)
- moved C4 1.61 mm to (298.0, 116.8)
- moved C6 1.61 mm to (292.1, 128.5)
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Routing:
- net Net-(LED54-Pad4): track 0.00 -> 402.7 mm, vias 0 -> 4
- net Net-(LED35-Pad4): track 0.00 -> 399.8 mm, vias 0 -> 4
- net Net-(LED89-Pad4): track 0.00 -> 397.1 mm, vias 0 -> 2
- net Net-(LED71-Pad4): track 0.00 -> 374.8 mm, vias 0 -> 2
- net Net-(LED16-Pad4): track 0.00 -> 318.5 mm, vias 0 -> 2
- net Net-(LED1-Pad2): track 0.00 -> 290.4 mm, vias 0 -> 1
- net COL1: track 0.00 -> 125.1 mm
- net COL2: track 0.00 -> 120.2 mm
- net COL15: track 0.00 -> 119.7 mm
- net COL14: track 0.00 -> 118.0 mm
- net COL5: track 0.00 -> 117.2 mm
- net COL10: track 0.00 -> 116.8 mm
- net COL9: track 0.00 -> 116.8 mm
- net COL12: track 0.00 -> 113.4 mm
- net ROT_A: track 0.00 -> 112.2 mm, vias 0 -> 4
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- added copper zone on In2.Cu, net +3V3
- added copper zone on In1.Cu, net GND
