File: thpd-kb01.kicad_pcb (KiCad board)
At the start: 4 copper layers, 388 x 116 mm, 344 parts, among them J1 USB_C_Receptacle_USB2.0, SW1 SW_Push, SW2 SW_SPDT, SW3 Rotary_Encoder_Switch, U1 XC6206PxxxMR, U2 USBLC6-2SC6, U3 NHD-C12832A1Z, U4 STM32F072C8Tx

Commit message: WIP
Routing:
- net ROT_SW_ROW: track 0.00 -> 5.41 mm
- net ROT_A: track 112.2 -> 108.2 mm

Commit message: All routing except row/col done.
Parts:
- moved SW1 35.5 mm to (273.9, 125.5), turned to 270 degrees
- moved C11 30.1 mm to (276.2, 127.3), turned to 90 degrees
- moved SW2 18.5 mm to (302.4, 147.4), turned to 90 degrees
- moved R5 13.6 mm to (297.5, 148.1), turned to 0 degrees
- moved C7 0.32 mm to (289.1, 121.7)
- moved C8 0.32 mm to (288.0, 121.7)
Routing:
- net ROW0: track 0.00 -> 375.9 mm
- net ROW1: track 0.00 -> 371.7 mm, vias 0 -> 6
- net ROW2: track 0.00 -> 369.2 mm, vias 0 -> 2
- net ROW4: track 0.00 -> 358.4 mm
- net ROW5: track 0.00 -> 345.3 mm
- net ROW3: track 0.00 -> 342.4 mm
- net Net-(C11-Pad1): track 40.5 -> 23.4 mm
- net COL13: track 83.3 -> 96.7 mm, vias 0 -> 1
- net Net-(R5-Pad1): track 29.4 -> 22.3 mm
- net Net-(D88-Pad2): track 0.00 -> 4.54 mm
- net Net-(D87-Pad2): track 0.00 -> 4.54 mm
- net Net-(D86-Pad2): track 0.00 -> 4.54 mm
- net Net-(D85-Pad2): track 0.00 -> 4.54 mm
- net Net-(D84-Pad2): track 0.00 -> 4.54 mm
- net Net-(D83-Pad2): track 0.00 -> 4.54 mm
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
Commit message: WIP
Parts:
- moved C11 99.2 mm to (357.3, 184.4)
- moved SW1 99.2 mm to (355.0, 182.6)
- moved R5 74.7 mm to (359.5, 189.8)
- moved SW2 74.7 mm to (364.4, 189.1)
- moved R10 71.0 mm to (321.4, 180.3), turned to 270 degrees
- moved U4 69.6 mm to (328.4, 183.7)
- moved C9 69.6 mm to (334.3, 186.7)
- moved C3 69.6 mm to (331.4, 176.8)
- moved C4 69.6 mm to (331.4, 177.9)
- moved C5 69.6 mm to (325.5, 190.8)
- moved C7 69.6 mm to (322.5, 182.8)
- moved C8 69.6 mm to (321.4, 182.8)
- moved C10 69.6 mm to (335.5, 186.7)
- moved C6 69.6 mm to (325.5, 189.6)
- moved U2 0.92 mm to (327.6, 95.1)
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Routing:
- net Net-(LED89-Pad4): track 397.1 -> 0.00 mm, vias 2 -> 0
- net Net-(LED1-Pad2): track 290.4 -> 0.00 mm, vias 1 -> 0
- net ROT_A: track 108.2 -> 0.00 mm, vias 4 -> 0
- net ROT_B: track 98.7 -> 0.00 mm, vias 4 -> 0
- net D_USB-: track 41.7 -> 92.2 mm, vias 0 -> 2
- net D_USB+: track 42.5 -> 91.5 mm, vias 0 -> 2
- net SPI1_SCK: track 73.7 -> 109.8 mm, vias 2 -> 4
- net SPI1_MOSI: track 75.2 -> 108.5 mm
- net LCD_CS: track 75.2 -> 107.7 mm
- net LCD_RST: track 75.6 -> 108.0 mm
- net LCD_A0: track 75.6 -> 107.0 mm
- net Net-(C11-Pad1): track 23.4 -> 0.00 mm
- net Net-(R5-Pad1): track 22.3 -> 0.00 mm
- net COL13: track 96.7 -> 110.9 mm, vias 1 -> 2
- net Net-(LED54-Pad4): track 402.7 -> 391.1 mm, vias 4 -> 2
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Other:
- rule trace_min: 0.2 -> 0.09
- rule via_min_drill: 0.3 -> 0.2

Commit message: WIP
Parts:
- moved SW2 63.7 mm to (301.1, 182.3), turned to 270 degrees
- moved R5 52.9 mm to (307.2, 181.6), turned to 180 degrees
- moved C11 37.3 mm to (320.6, 177.5), turned to 0 degrees
- moved SW1 33.4 mm to (322.4, 175.2), turned to 180 degrees
- moved R10 12.2 mm to (333.2, 177.2)
- moved C8 11.5 mm to (331.1, 176.7), turned to 180 degrees
- moved C3 11.4 mm to (337.1, 186.7), turned to 90 degrees
- moved C5 10.3 mm to (323.1, 180.8), turned to 270 degrees
- moved C7 9.95 mm to (331.1, 177.8), turned to 180 degrees
- moved C4 9.93 mm to (336.0, 186.7), turned to 90 degrees
- moved C10 9.26 mm to (327.2, 190.8), turned to 0 degrees
- moved C6 8.88 mm to (324.3, 180.8), turned to 270 degrees
- moved C9 7.67 mm to (327.2, 189.6), turned to 0 degrees
- moved U4 1.77 mm to (330.2, 183.7), turned to 270 degrees
Routing:
- net Net-(LED89-Pad4): track 0.00 -> 377.0 mm
- net Net-(R5-Pad1): track 0.00 -> 19.0 mm
- net LCD_CS: track 107.7 -> 89.5 mm, vias 2 -> 1
- net LCD_RST: track 108.0 -> 91.0 mm, vias 2 -> 1
- net SPI1_SCK: track 109.8 -> 93.1 mm, vias 4 -> 2
- net Net-(C11-Pad1): track 0.00 -> 15.2 mm
- net LCD_A0: track 107.0 -> 93.3 mm, vias 2 -> 1
- net SPI1_MOSI: track 108.5 -> 95.3 mm, vias 2 -> 1
- net D_USB+: track 91.5 -> 89.5 mm
- net Net-(R5-Pad2): track 2.01 -> 3.21 mm
- net D_USB-: track 92.2 -> 91.2 mm
- net /led_matrix/DIN: track 2.91 -> 1.95 mm
- net Net-(LED32-Pad4): vias 0 -> 2
- net Net-(LED86-Pad4): vias 0 -> 2
- net Net-(LED51-Pad4): vias 0 -> 2
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
Commit message: WIP
Parts:
- moved R5 4.48 mm to (309.0, 177.5)
- moved SW2 4.48 mm to (302.9, 178.2)
Routing:
- net ROT_A: track 0.00 -> 183.4 mm, vias 0 -> 2
- net ROT_B: track 0.00 -> 169.4 mm, vias 0 -> 2
- net ROW5: track 345.3 -> 358.4 mm
- net ROW4: track 358.4 -> 364.9 mm
- net Net-(R5-Pad1): track 19.0 -> 20.4 mm
Changed lines of the file:
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@@
     (thickness 1.6)
     (drawings 6)
-    (tracks 1164)
+    (tracks 1206)
     (zones 0)
     (modules 344)
@@
   )
   (module thpd-kb01-custom:SW_SPDT_K3-1296S-E1 (layer B.Cu)
-    (at 301.093751 182.3475 270)
+    (at 302.893751 178.2475 270)
     (fp_text reference SW2 (at 0 -4 90) (layer B.SilkS)
       (effects (font (size 1 1) (thickness 0.15)) (justify mirror))
@@
   )
   (module Resistor_SMD:R_0603_1608Metric (layer B.Cu)
-    (at 307.2 181.6 180)
+    (at 309 177.5 180)
     (descr "Resistor SMD 0603 (1608 Metric), square (rectangular) end terminal, IPC_7351 nominal, (Body size source: IPC-SM-782 page 72, https://www.pcb-3d.com/wordpress/wp-content/uploads/ipc-sm-782a_amendment_1_and_2.pdf), generated with kicad-footprint-generator")
     (tags resistor)
@@
   (segment (start 360.45 98.07) (end 360.28 97.9) (width 0.3) (layer B.Cu) (net 14) (status 30))
   (segment (start 360.45 100.0125) (end 360.45 98.07) (width 0.3) (layer B.Cu) (net 14) (status 30))
+  (segment (start 385.425 97.75) (end 384.175 96.5) (width 0.3) (layer B.Cu) (net 15))
+  (segment (start 385.47 97.75) (end 385.425 97.75) (width 0.3) (layer B.Cu) (net 15))
+  (via (at 334.6 191.1) (size 0.8) (drill 0.4) (layers F.Cu B.Cu) (net 15))
+  (segment (start 334.6 191.1) (end 333.1 191.1) (width 0.3) (layer F.Cu) (net 15))
+  (segment (start 386 191.1) (end 334.6 191.1) (width 0.3) (layer B.Cu) (net 15))
+  (segment (start 399.6 102.1) (end 399.6 177.5) (width 0.3) (layer B.Cu) (net 15))
+  (segment (start 396.6 99.1) (end 399.6 102.1) (width 0.3) (layer B.Cu) (net 15))
+  (segment (start 386.51 99.1) (end 396.6 99.1) (width 0.3) (layer B.Cu) (net 15))
+  (segment (start 385.47 98.06) (end 386.51 99.1) (width 0.3) (layer B.Cu) (net 15))
+  (segment (start 399.6 177.5) (end 386 191.1) (width 0.3) (layer B.Cu) (net 15))
+  (segment (start 385.47 97.75) (end 385.47 98.06) (width 0.3) (layer B.Cu) (net 15))
+  (via (at 332.8 191.1) (size 0.8) (drill 0.4) (layers F.Cu B.Cu) (net 15))
+  (segment (start 333.1 191.1) (end 332.8 191.1) (width 0.3) (layer F.Cu) (net 15))
+  (segment (start 332.149999 190.449999) (end 332.8 191.1) (width 0.3) (layer B.Cu) (net 15))
+  (segment (start 332.149999 189.439999) (end 332.149999 190.449999) (width 0.3) (layer B.Cu) (net 15))
+  (segment (start 332.4375 189.152498) (end 332.149999 189.439999) (width 0.3) (layer B.Cu) (net 15))
+  (segment (start 332.4375 187.875) (end 332.4375 189.152498) (width 0.3) (layer B.Cu) (net 15))
+  (segment (start 385.375 85.6) (end 384.175 86.8) (width 0.3) (layer B.Cu) (net 16))
+  (segment (start 385.445 85.6) (end 385.375 85.6) (width 0.3) (layer B.Cu) (net 16))
+  (segment (start 379.39374 94.134072) (end 385.059668 99.8) (width 0.3) (layer B.Cu) (net 16))
+  (segment (start 381.784668 86.8) (end 379.39374 89.190928) (width 0.3) (layer B.Cu) (net 16))
+  (segment (start 379.39374 89.190928) (end 379.39374 94.134072) (width 0.3) (layer B.Cu) (net 16))
+  (segment (start 384.175 86.8) (end 381.784668 86.8) (width 0.3) (layer B.Cu) (net 16))
+  (segment (start 385.059668 99.8) (end 396.1 99.8) (width 0.3) (layer B.Cu) (net 16))
+  (segment (start 398.9 102.6) (end 398.9 177.1) (width 0.3) (layer B.Cu) (net 16))
+  (segment (start 396.1 99.8) (end 398.9 102.6) (width 0.3) (layer B.Cu) (net 16))
+  (segment (start 398.9 177.1) (end 395.8 180.2) (width 0.3) (layer B.Cu) (net 16))
+  (via (at 334.6 190.1) (size 0.8) (drill 0.4) (layers F.Cu B.Cu) (net 16))
+  (segment (start 385.9 190.1) (end 334.6 190.1) (width 0.3) (layer B.Cu) (net 16))
+  (segment (start 395.8 180.2) (end 385.9 190.1) (width 0.3) (layer B.Cu) (net 16))
+  (via (at 332.9 189.8) (size 0.8) (drill 0.4) (layers F.Cu B.Cu) (net 16))
+  (segment (start 333.2 190.1) (end 332.9 189.8) (width 0.3) (layer F.Cu) (net 16))
+  (segment (start 334.6 190.1) (end 333.2 190.1) (width 0.3) (layer F.Cu) (net 16))
+  (segment (start 332.9375 189.7625) (end 332.9375 187.875) (width 0.3) (layer B.Cu) (net 16))
+  (segment (start 332.9 189.8) (end 332.9375 189.7625) (width 0.3) (layer B.Cu) (net 16))
   (segment (start 23.01875 89.05875) (end 23.01875 93.6) (width 0.3) (layer B.Cu) (net 17) (status 30))
   (segment (start 42.06875 89.05875) (end 42.06875 93.6) (width 0.3) (layer B.Cu) (net 18) (status 30))
@@
   (segment (start 327.8508 185.9) (end 328.9375 186.9867) (width 0.175006) (layer B.Cu) (net 126))
   (segment (start 303.171251 181.6) (end 303.168751 181.5975) (width 0.3) (layer B.Cu) (net 127))
-  (segment (start 306.375 181.6) (end 303.171251 181.6) (width 0.3) (layer B.Cu) (net 127))
-  (segment (start 308.425 181.6) (end 308.025 181.6) (width 0.3) (layer B.Cu) (net 128))
-  (segment (start 310.325 183.5) (end 308.425 181.6) (width 0.3) (layer B.Cu) (net 128))
-  (segment (start 317.2 183.5) (end 310.325 183.5) (width 0.3) (layer B.Cu) (net 128))
-  (segment (start 317.7375 182.9625) (end 317.2 183.5) (width 0.3) (layer B.Cu) (net 128))
-  (segment (start 326.025 182.9625) (end 317.7375 182.9625) (width 0.3) (layer B.Cu) (net 128))
+  (segment (start 308.175 177.5) (end 304.971251 177.5) (width 0.3) (layer B.Cu) (net 127))
+  (segment (start 309.825 179.525) (end 309.825 177.5) (width 0.3) (layer B.Cu) (net 128))
+  (segment (start 314.2 183.9) (end 309.825 179.525) (width 0.3) (layer B.Cu) (net 128))
+  (segment (start 316.4 183.9) (end 314.2 183.9) (width 0.3) (layer B.Cu) (net 128))
+  (segment (start 317.3375 182.9625) (end 316.4 183.9) (width 0.3) (layer B.Cu) (net 128))
+  (segment (start 326.025 182.9625) (end 317.3375 182.9625) (width 0.3) (layer B.Cu) (net 128))
   (segment (start 383.0125 94.85) (end 381.825 93.6625) (width 0.3) (layer B.Cu) (net 129) (status 20))
   (segment (start 384.175 94.85) (end 383.0125 94.85) (width 0.3) (layer B.Cu) (net 129) (status 10))
@@
   (segment (start 263.525 173.1) (end 289.71875 173.1) (width 0.3) (layer B.Cu) (net 243) (status 30))
   (segment (start 289.71875 173.1) (end 308.76875 173.1) (width 0.3) (layer B.Cu) (net 243) (status 30))
-  (segment (start 308.76875 173.1) (end 332.58125 173.1) (width 0.3) (layer B.Cu) (net 243) (status 30))
   (segment (start 332.58125 173.1) (end 351.63125 173.1) (width 0.3) (layer B.Cu) (net 243) (status 30))
   (segment (start 351.63125 173.1) (end 370.68125 173.1) (width 0.3) (layer B.Cu) (net 243) (status 30))
   (segment (start 384.84375 173.1) (end 389.73125 168.2125) (width 0.3) (layer B.Cu) (net 243) (status 20))
   (segment (start 370.68125 173.1) (end 384.84375 173.1) (width 0.3) (layer B.Cu) (net 243) (status 10))
+  (segment (start 329.9375 179.55) (end 329.9375 173.1625) (width 0.3) (layer B.Cu) (net 243))
+  (segment (start 330 173.1) (end 332.58125 173.1) (width 0.3) (layer B.Cu) (net 243))
+  (segment (start 329.9375 173.1625) (end 330 173.1) (width 0.3) (layer B.Cu) (net 243))
+  (segment (start 308.76875 173.1) (end 330 173.1) (width 0.3) (layer B.Cu) (net 243))
   (segment (start 25.4 192.15) (end 49.2125 192.15) (width 0.3) (layer B.Cu) (net 244) (status 30))
   (segment (start 49.2125 192.15) (end 73.025 192.15) (width 0.3) (layer B.Cu) (net 244) (status 30))
@@
   (segment (start 270.66875 192.15) (end 289.71875 192.15) (width 0.3) (layer B.Cu) (net 244) (status 30))
   (segment (start 289.71875 192.15) (end 308.76875 192.15) (width 0.3) (layer B.Cu) (net 244) (status 30))
-  (segment (start 308.76875 192.15) (end 342.10625 192.15) (width 0.3) (layer B.Cu) (net 244) (status 30))
   (segment (start 342.10625 192.15) (end 370.68125 192.15) (width 0.3) (layer B.Cu) (net 244) (status 30))
+  (segment (start 332.4375 186.036442) (end 333.65 187.248942) (width 0.3) (layer B.Cu) (net 244))
+  (segment (start 332.4375 179.55) (end 332.4375 186.036442) (width 0.3) (layer B.Cu) (net 244))
+  (segment (start 333.65 187.248942) (end 333.65 192.15) (width 0.3) (layer B.Cu) (net 244))
+  (segment (start 333.65 192.15) (end 342.10625 192.15) (width 0.3) (layer B.Cu) (net 244))
+  (segment (start 308.76875 192.15) (end 333.65 192.15) (width 0.3) (layer B.Cu) (net 244))
   (segment (start 29.36875 92.673748) (end 27.428749 94.613749) (width 0.3) (layer F.Cu) (net 245))
   (segment (start 27.428749 103.628749) (end 29.36875 105.56875) (width 0.3) (layer F.Cu) (net 245) (status 20))

Commit message: Routing of rows and columns done.
Parts:
- moved C11 5.59 mm to (315.1, 178.5)
- moved SW1 5.59 mm to (316.9, 176.2)
Connections:
- net Net-(C11-Pad1) renamed NRST
- net Net-(R5-Pad1) renamed BOOT0
- U4 pad 11: ROW5 -> (no net)
- U4 pad 18: COL9 -> COL15
- U4 pad 19: COL10 -> COL16
- U4 pad 20: COL11 -> COL17
- U4 pad 21: COL12 -> COL18
- U4 pad 22: COL13 -> ROT_A
- U4 pad 25: ROT_A -> ROT_B
- U4 pad 26: ROT_B -> ROW5
- U4 pad 27: COL14 -> COL0
- U4 pad 28: COL15 -> COL1
- U4 pad 29: COL16 -> COL2
- U4 pad 30: COL17 -> COL3
- U4 pad 31: COL18 -> COL4
- U4 pad 34: (no net) -> COL5
- U4 pad 37: COL0 -> COL6
- U4 pad 38: COL1 -> COL7
- U4 pad 39: COL2 -> COL8
- U4 pad 40: COL3 -> COL9
- U4 pad 41: COL4 -> COL10
- U4 pad 42: COL5 -> COL11
- U4 pad 43: COL6 -> COL12
- U4 pad 45: COL7 -> COL13
- U4 pad 46: COL8 -> COL14
Routing:
- net Net-(LED1-Pad2): track 0.00 -> 401.5 mm, vias 0 -> 3
- net COL0: track 110.2 -> 432.9 mm, vias 0 -> 1
- net COL1: track 125.1 -> 422.4 mm, vias 0 -> 1
- net COL2: track 120.2 -> 392.2 mm, vias 0 -> 1
- net COL3: track 95.7 -> 342.9 mm, vias 0 -> 1
- net COL4: track 95.7 -> 324.8 mm, vias 0 -> 1
- net COL5: track 117.2 -> 313.7 mm, vias 0 -> 1
- net COL6: track 95.7 -> 277.6 mm, vias 0 -> 1
- net COL7: track 95.7 -> 257.9 mm, vias 0 -> 1
- net COL8: track 95.7 -> 238.6 mm, vias 0 -> 1
- net COL9: track 116.8 -> 228.1 mm
- net ROW0: track 375.9 -> 470.0 mm, vias 0 -> 2
- net COL10: track 116.8 -> 208.2 mm
- net COL11: track 110.9 -> 182.3 mm
- net COL18: track 82.2 -> 150.5 mm, vias 0 -> 2
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
Commit message: All routing complete.
Routing:
- net GND: track 32.7 -> 265.5 mm, vias 8 -> 114
- net +3V3: track 16.9 -> 135.2 mm, vias 2 -> 109
- net NRST: track 20.3 -> 33.7 mm, vias 0 -> 2
