File: thpd-kb01.sch (KiCad schematic (older format))
At the start: 16 parts

Commit message: wip
Parts:
- C1, C2, C3, C4, C5, C6, C7: renamed from C?; footprint (none) -> Capacitor_SMD:C_0805_2012Metric
- F1: renamed from F?; footprint (none) -> Fuse:Fuse_1206_3216Metric
- R1, R2, R3, R4: renamed from R?; footprint (none) -> Resistor_SMD:R_0805_2012Metric
- SW1: renamed from SW?; footprint (none) -> random-keyboard-parts:SKQG-1155865
- USB1: renamed from USB?; footprint (none) -> random-keyboard-parts:Molex-0548190589
- Y1: renamed from Y?; footprint (none) -> Crystal:Crystal_SMD_3225-4Pin_3.2x2.5mm
- gave numbers to parts that had none: 1
Other:
- moved on the sheet: C1, C2, C3, C4, C5, C6, C7, R1, R2, R3, R4, SW1

Commit message: Switch USB B to USB C
Parts:
- removed USB1: Molex-0548190589, random-keyboard-parts:Molex-0548190589, symbol random-keyboard-parts:Molex-0548190589
- added J1: USB_C_Receptacle_USB2.0, Connector_USB:USB_C_Receptacle_JAE_DX07S024WJ3R400, symbol Connector:USB_C_Receptacle_USB2.0
- added R5, R6: 5.1k, Resistor_SMD:R_0805_2012Metric, symbol Device:R_Small
Connections:
- wire segments 51 -> 61
- no-connect marks 0 -> 2
Other:
- moved on the sheet: F1
Changed lines of the file:
@@
 Wire Wire Line
 	3700 4850 4150 4850
-$Comp
-L random-keyboard-parts:Molex-0548190589 USB1
-U 1 1 61778ED3
-P 1250 6350
-F 0 "USB1" V 1787 6317 60  0000 C CNN
-F 1 "Molex-0548190589" V 1681 6317 60  0000 C CNN
-F 2 "random-keyboard-parts:Molex-0548190589" H 1250 6350 60  0001 C CNN
-F 3 "" H 1250 6350 60  0001 C CNN
-	1    1250 6350
-	0    -1   -1   0
-$EndComp
-$Comp
-L Device:Polyfuse_Small F1
-U 1 1 61779F39
-P 2150 6150
-F 0 "F1" V 1945 6150 50  0000 C CNN
-F 1 "500mA" V 2036 6150 50  0000 C CNN
-F 2 "Fuse:Fuse_1206_3216Metric" H 2200 5950 50  0001 L CNN
-F 3 "~" H 2150 6150 50  0001 C CNN
-	1    2150 6150
-	0    1    1    0
-$EndComp
-Wire Wire Line
-	1550 6150 1800 6150
-$Comp
-L power:+5V #PWR06
-U 1 1 6177BB60
-P 2650 6150
-F 0 "#PWR06" H 2650 6000 50  0001 C CNN
-F 1 "+5V" H 2665 6323 50  0000 C CNN
-F 2 "" H 2650 6150 50  0001 C CNN
-F 3 "" H 2650 6150 50  0001 C CNN
-	1    2650 6150
-	1    0    0    -1
-$EndComp
-Wire Wire Line
-	2250 6150 2650 6150
-$Comp
-L power:VCC #PWR04
-U 1 1 6177DA57
-P 1800 6150
-F 0 "#PWR04" H 1800 6000 50  0001 C CNN
-F 1 "VCC" H 1815 6323 50  0000 C CNN
-F 2 "" H 1800 6150 50  0001 C CNN
-F 3 "" H 1800 6150 50  0001 C CNN
-	1    1800 6150
-	1    0    0    -1
-$EndComp
-Connection ~ 1800 6150
-Wire Wire Line
-	1800 6150 2050 6150
-Text GLabel 1700 6350 2    50   Input ~ 0
-D+
-Text GLabel 1700 6250 2    50   Input ~ 0
-D-
-Wire Wire Line
-	1700 6250 1550 6250
-Wire Wire Line
-	1550 6350 1700 6350
-$Comp
-L power:GND #PWR03
-U 1 1 61781036
-P 1750 6550
-F 0 "#PWR03" H 1750 6300 50  0001 C CNN
-F 1 "GND" H 1755 6377 50  0000 C CNN
-F 2 "" H 1750 6550 50  0001 C CNN
-F 3 "" H 1750 6550 50  0001 C CNN
-	1    1750 6550
-	1    0    0    -1
-$EndComp
-Wire Wire Line
-	1750 6550 1550 6550
 Wire Wire Line
 	4850 3650 4900 3650
@@
 F25 "COL17" I L 6550 3900 50
 $EndSheet
+$Comp
+L power:GND #PWR03
+U 1 1 61781036
+P 1050 7200
+F 0 "#PWR03" H 1050 6950 50  0001 C CNN
+F 1 "GND" H 1055 7027 50  0000 C CNN
+F 2 "" H 1050 7200 50  0001 C CNN
+F 3 "" H 1050 7200 50  0001 C CNN
+	1    1050 7200
+	1    0    0    -1
+$EndComp
+Text GLabel 2200 6200 2    50   Input ~ 0
+D-
+Text GLabel 2200 6300 2    50   Input ~ 0
+D+
+Wire Wire Line
+	2200 5600 2450 5600
+$Comp
+L power:VCC #PWR04
+U 1 1 6177DA57
+P 2200 5600
+F 0 "#PWR04" H 2200 5450 50  0001 C CNN
+F 1 "VCC" H 2215 5773 50  0000 C CNN
+F 2 "" H 2200 5600 50  0001 C CNN
+F 3 "" H 2200 5600 50  0001 C CNN
+	1    2200 5600
+	1    0    0    -1
+$EndComp
+Wire Wire Line
+	2650 5600 3050 5600
+$Comp
+L power:+5V #PWR06
+U 1 1 6177BB60
+P 3050 5600
+F 0 "#PWR06" H 3050 5450 50  0001 C CNN
+F 1 "+5V" H 3065 5773 50  0000 C CNN
+F 2 "" H 3050 5600 50  0001 C CNN
+F 3 "" H 3050 5600 50  0001 C CNN
+	1    3050 5600
+	1    0    0    -1
+$EndComp
+$Comp
+L Device:Polyfuse_Small F1
+U 1 1 61779F39
+P 2550 5600
+F 0 "F1" V 2345 5600 50  0000 C CNN
+F 1 "500mA" V 2436 5600 50  0000 C CNN
+F 2 "Fuse:Fuse_1206_3216Metric" H 2600 5400 50  0001 L CNN
+F 3 "~" H 2550 5600 50  0001 C CNN
+	1    2550 5600
+	0    1    1    0
+$EndComp
+$Comp
+L Connector:USB_C_Receptacle_USB2.0 J1
+U 1 1 61899044
+P 1350 6200
+F 0 "J1" H 1457 7067 50  0000 C CNN
+F 1 "USB_C_Receptacle_USB2.0" H 1457 6976 50  0000 C CNN
+F 2 "Connector_USB:USB_C_Receptacle_JAE_DX07S024WJ3R400" H 1500 6200 50  0001 C CNN
+F 3 "https://www.usb.org/sites/default/files/documents/usb_type-c.zip" H 1500 6200 50  0001 C CNN
+	1    1350 6200
+	1    0    0    -1
+$EndComp
+Wire Wire Line
+	1350 7100 1050 7100
+Wire Wire Line
+	1050 7200 1050 7100
+Connection ~ 1050 7100
+Wire Wire Line
+	1950 5600 2200 5600
+Connection ~ 2200 5600
+Wire Wire Line
+	2200 6200 1950 6200
+Wire Wire Line
+	1950 6100 1950 6200
+Connection ~ 1950 6200
+Wire Wire Line
+	1950 6400 1950 6300
+Wire Wire Line
+	1950 6300 2200 6300
+Connection ~ 1950 6300
+NoConn ~ 1950 6700
+NoConn ~ 1950 6800
+$Comp
+L Device:R_Small R5
+U 1 1 618A7116
+P 2600 6000
+F 0 "R5" H 2541 5954 50  0000 R CNN
+F 1 "5.1k" H 2541 6045 50  0000 R CNN
+F 2 "Resistor_SMD:R_0805_2012Metric" H 2600 6000 50  0001 C CNN
+F 3 "~" H 2600 6000 50  0001 C CNN
+	1    2600 6000
+	-1   0    0    1
+$EndComp
+$Comp
+L Device:R_Small R6
+U 1 1 618A870D
+P 2900 6000
+F 0 "R6" H 2959 6046 50  0000 L CNN
+F 1 "5.1k" H 2959 5955 50  0000 L CNN
+F 2 "Resistor_SMD:R_0805_2012Metric" H 2900 6000 50  0001 C CNN
+F 3 "~" H 2900 6000 50  0001 C CNN
+	1    2900 6000
+	1    0    0    -1
+$EndComp
+Wire Wire Line
+	1950 5900 2600 5900
+Wire Wire Line
+	1950 5800 2900 5800
+Wire Wire Line
+	2600 6100 2600 7100
+Wire Wire Line
+	2600 7100 1350 7100
+Connection ~ 1350 7100
+Connection ~ 2600 7100
+Wire Wire Line
+	2900 5800 2900 5900
+Wire Wire Line
+	2900 6100 2900 7100
+Wire Wire Line
+	2900 7100 2600 7100
 $EndSCHEMATC

Commit message: wip
Parts:
- J1: footprint Connector_USB:USB_C_Receptacle_JAE_DX07S024WJ3R400 -> Connector_USB:USB_C_Receptacle_HRO_TYPE-C-31-M-12
- SW1: footprint random-keyboard-parts:SKQG-1155865 -> random-keyboard-parts:SKQGADE010
Changed lines of the file:
@@
 F 0 "SW1" H 3350 1835 50  0000 C CNN
 F 1 "SW_Push" H 3350 1744 50  0000 C CNN
-F 2 "random-keyboard-parts:SKQG-1155865" H 3350 1750 50  0001 C CNN
+F 2 "random-keyboard-parts:SKQGADE010" H 3350 1750 50  0001 C CNN
 F 3 "~" H 3350 1750 50  0001 C CNN
 	1    3350 1550
@@
 F 0 "J1" H 1457 7067 50  0000 C CNN
 F 1 "USB_C_Receptacle_USB2.0" H 1457 6976 50  0000 C CNN
-F 2 "Connector_USB:USB_C_Receptacle_JAE_DX07S024WJ3R400" H 1500 6200 50  0001 C CNN
+F 2 "Connector_USB:USB_C_Receptacle_HRO_TYPE-C-31-M-12" H 1500 6200 50  0001 C CNN
 F 3 "https://www.usb.org/sites/default/files/documents/usb_type-c.zip" H 1500 6200 50  0001 C CNN
 	1    1350 6200

Commit message: Switch to STM32F072CBT6 MCU
Parts:
- removed C1, C2, C3: 0.1uF, Capacitor_SMD:C_0805_2012Metric, symbol Device:C_Small
- removed C4: 10uF, Capacitor_SMD:C_0805_2012Metric, symbol Device:C_Small
- removed C5, C6: 22pF, Capacitor_SMD:C_0805_2012Metric, symbol Device:C_Small
- removed C7: 1uF, Capacitor_SMD:C_0805_2012Metric, symbol Device:C_Small
- removed R1, R2: 22, Resistor_SMD:R_0805_2012Metric, symbol Device:R_Small
- removed R3, R4: 10k, Resistor_SMD:R_0805_2012Metric, symbol Device:R_Small
- removed SW1: SW_Push, random-keyboard-parts:SKQGADE010, symbol Switch:SW_Push
- removed U1: ATmega32U4-AU, Package_QFP:TQFP-44_10x10mm_P0.8mm, symbol MCU_Microchip_ATmega:ATmega32U4-AU
- removed Y1: 16MHz, Crystal:Crystal_SMD_3225-4Pin_3.2x2.5mm, symbol Device:Crystal_GND24_Small
- added C? (x5): 100nF, symbol Device:C_Small
- added C? (x2): 4.7uF, symbol Device:C_Small
- added C? (x3): 1uF, symbol Device:C_Small
- added C?: 10nF, symbol Device:C_Small
- added R?: 10k, symbol Device:R_Small
- added R? (x2): 22, symbol Device:R_Small
- added SW?: SW_SPDT, symbol Switch:SW_SPDT
- added SW?: SW_Push, symbol Switch:SW_Push
- added U?: STM32F072C8Tx, Package_QFP:LQFP-48_7x7mm_P0.5mm, symbol MCU_ST_STM32F0:STM32F072C8Tx
- added U?: USBLC6-2SC6, Package_TO_SOT_SMD:SOT-23-6, symbol Power_Protection:USBLC6-2SC6
- added U?: XC6206PxxxMR, Package_TO_SOT_SMD:SOT-23, symbol Regulator_Linear:XC6206PxxxMR
Connections:
- net labels added: +3.3V, DCONN+, DCONN-
- net labels removed: VCC
- wire segments 61 -> 70
Other:
- moved on the sheet: F1

Commit message: re-annotate symbols
Parts:
- gave numbers to parts that had none: 19
- renumbered R5 to R2, R6 to R3
Changed lines of the file:
@@
 $EndSheet
 $Comp
-L power:GND #PWR03
+L power:GND #PWR01
 U 1 1 61781036
 P 1050 7200
-F 0 "#PWR03" H 1050 6950 50  0001 C CNN
+F 0 "#PWR01" H 1050 6950 50  0001 C CNN
 F 1 "GND" H 1055 7027 50  0000 C CNN
 F 2 "" H 1050 7200 50  0001 C CNN
@@
 D+
 $Comp
-L power:+5V #PWR06
+L power:+5V #PWR08
 U 1 1 6177BB60
 P 4150 5850
-F 0 "#PWR06" H 4150 5700 50  0001 C CNN
+F 0 "#PWR08" H 4150 5700 50  0001 C CNN
 F 1 "+5V" H 4165 6023 50  0000 C CNN
 F 2 "" H 4150 5850 50  0001 C CNN
@@
 NoConn ~ 1950 6800
 $Comp
-L Device:R_Small R5
+L Device:R_Small R2
 U 1 1 618A7116
 P 2600 6000
-F 0 "R5" H 2541 5954 50  0000 R CNN
+F 0 "R2" H 2541 5954 50  0000 R CNN
 F 1 "5.1k" H 2541 6045 50  0000 R CNN
 F 2 "Resistor_SMD:R_0805_2012Metric" H 2600 6000 50  0001 C CNN
@@
 $EndComp
 $Comp
-L Device:R_Small R6
+L Device:R_Small R3
 U 1 1 618A870D
 P 2900 6000
-F 0 "R6" H 2959 6046 50  0000 L CNN
+F 0 "R3" H 2959 6046 50  0000 L CNN
 F 1 "5.1k" H 2959 5955 50  0000 L CNN
 F 2 "Resistor_SMD:R_0805_2012Metric" H 2900 6000 50  0001 C CNN
@@
 	2900 7100 2600 7100
 $Comp
-L MCU_ST_STM32F0:STM32F072C8Tx U?
+L MCU_ST_STM32F0:STM32F072C8Tx U1
 U 1 1 618DB153
 P 3650 2950
-F 0 "U?" H 3600 1361 50  0000 C CNN
+F 0 "U1" H 3600 1361 50  0000 C CNN
 F 1 "STM32F072C8Tx" H 3600 1270 50  0000 C CNN
 F 2 "Package_QFP:LQFP-48_7x7mm_P0.5mm" H 3050 1550 50  0001 R CNN
@@
 	3750 1450 3650 1450
 $Comp
-L power:GND #PWR?
+L power:GND #PWR07
 U 1 1 618DCDD4
 P 3450 4750
-F 0 "#PWR?" H 3450 4500 50  0001 C CNN
+F 0 "#PWR07" H 3450 4500 50  0001 C CNN
 F 1 "GND" H 3455 4577 50  0000 C CNN
 F 2 "" H 3450 4750 50  0001 C CNN
@@
 	5400 5700 5600 5700
 $Comp
-L Power_Protection:USBLC6-2SC6 U?
+L Power_Protection:USBLC6-2SC6 U2
 U 1 1 61991CC6
 P 4150 6350
-F 0 "U?" H 4450 6000 50  0000 C CNN
+F 0 "U2" H 4450 6000 50  0000 C CNN
 F 1 "USBLC6-2SC6" H 4500 5900 50  0000 C CNN
 F 2 "Package_TO_SOT_SMD:SOT-23-6" H 4150 5850 50  0001 C CNN
@@
 DCONN+
 $Comp
-L power:GND #PWR?
+L power:GND #PWR09
 U 1 1 619952B6
 P 4150 6850
-F 0 "#PWR?" H 4150 6600 50  0001 C CNN
+F 0 "#PWR09" H 4150 6600 50  0001 C CNN
 F 1 "GND" H 4155 6677 50  0000 C CNN
 F 2 "" H 4150 6850 50  0001 C CNN
@@
 Connection ~ 1950 6200
 $Comp
-L Device:R_Small R?
+L Device:R_Small R5
 U 1 1 61997E5C
 P 4650 3850
-F 0 "R?" V 4454 3850 50  0000 C CNN
+F 0 "R5" V 4454 3850 50  0000 C CNN
 F 1 "22" V 4545 3850 50  0000 C CNN
 F 2 "" H 4650 3850 50  0001 C CNN
@@
 $EndComp
 $Comp
-L Device:R_Small R?
+L Device:R_Small R4
 U 1 1 619987AC
 P 4400 3950
-F 0 "R?" V 4204 3950 50  0000 C CNN
+F 0 "R4" V 4204 3950 50  0000 C CNN
 F 1 "22" V 4295 3950 50  0000 C CNN
 F 2 "" H 4400 3950 50  0001 C CNN
@@
 	4800 3850 4750 3850
 $Comp
-L power:+5V #PWR?
+L power:+5V #PWR04
 U 1 1 6199B61D
 P 2100 5600
-F 0 "#PWR?" H 2100 5450 50  0001 C CNN
+F 0 "#PWR04" H 2100 5450 50  0001 C CNN
 F 1 "+5V" H 2115 5773 50  0000 C CNN
 F 2 "" H 2100 5600 50  0001 C CNN
@@
 	2100 5600 1950 5600
 $Comp
-L power:+3.3V #PWR?
+L power:+3.3V #PWR06
 U 1 1 6199CAF2
 P 3450 1300
-F 0 "#PWR?" H 3450 1150 50  0001 C CNN
+F 0 "#PWR06" H 3450 1150 50  0001 C CNN
 F 1 "+3.3V" H 3465 1473 50  0000 C CNN
 F 2 "" H 3450 1300 50  0001 C CNN
@@
 $EndComp
 $Comp
-L Regulator_Linear:XC6206PxxxMR U?
+L Regulator_Linear:XC6206PxxxMR U3
 U 1 1 619BA934
 P 6250 5700
-F 0 "U?" H 6250 5942 50  0000 C CNN
+F 0 "U3" H 6250 5942 50  0000 C CNN
 F 1 "XC6206PxxxMR" H 6250 5851 50  0000 C CNN
 F 2 "Package_TO_SOT_SMD:SOT-23" H 6250 5925 50  0001 C CIN
@@
 $EndComp
 $Comp
-L Device:C_Small C?
+L Device:C_Small C2
 U 1 1 619BB4C8
 P 5600 5800
-F 0 "C?" H 5692 5846 50  0000 L CNN
+F 0 "C2" H 5692 5846 50  0000 L CNN
 F 1 "1uF" H 5692 5755 50  0000 L CNN
 F 2 "" H 5600 5800 50  0001 C CNN
@@
 Connection ~ 5600 5700
 $Comp
-L power:+5V #PWR?
+L power:+5V #PWR010
 U 1 1 619BD9A6
 P 5000 5700
-F 0 "#PWR?" H 5000 5550 50  0001 C CNN
+F 0 "#PWR010" H 5000 5550 50  0001 C CNN
 F 1 "+5V" H 5015 5873 50  0000 C CNN
 F 2 "" H 5000 5700 50  0001 C CNN
@@
 	5000 5700 5200 5700
 $Comp
-L power:GND #PWR?
+L power:GND #PWR011
 U 1 1 619BE6C8
 P 6250 6100
-F 0 "#PWR?" H 6250 5850 50  0001 C CNN
+F 0 "#PWR011" H 6250 5850 50  0001 C CNN
 F 1 "GND" H 6255 5927 50  0000 C CNN
 F 2 "" H 6250 6100 50  0001 C CNN
@@
 Connection ~ 6250 6000
 $Comp
-L Device:C_Small C?
+L Device:C_Small C3
 U 1 1 619BF843
 P 6700 5800
-F 0 "C?" H 6792 5846 50  0000 L CNN
+F 0 "C3" H 6792 5846 50  0000 L CNN
 F 1 "1uF" H 6792 5755 50  0000 L CNN
 F 2 "" H 6700 5800 50  0001 C CNN
@@
 $EndComp
 $Comp
-L power:+3.3V #PWR?
+L power:+3.3V #PWR012
 U 1 1 619C029E
 P 7050 5700
-F 0 "#PWR?" H 7050 5550 50  0001 C CNN
+F 0 "#PWR012" H 7050 5550 50  0001 C CNN
 F 1 "+3.3V" H 7065 5873 50  0000 C CNN
 F 2 "" H 7050 5700 50  0001 C CNN
@@
 	6700 6000 6250 6000
 $Comp
-L power:+3.3V #PWR?
+L power:+3.3V #PWR02
 U 1 1 6193E995
 P 1350 1650
-F 0 "#PWR?" H 1350 1500 50  0001 C CNN
+F 0 "#PWR02" H 1350 1500 50  0001 C CNN
 F 1 "+3.3V" H 1365 1823 50  0000 C CNN
 F 2 "" H 1350 1650 50  0001 C CNN
@@
 $EndComp
 $Comp
-L Switch:SW_SPDT SW?
+L Switch:SW_SPDT SW1
 U 1 1 6193D42E
 P 1650 1850
-F 0 "SW?" H 1650 1525 50  0000 C CNN
+F 0 "SW1" H 1650 1525 50  0000 C CNN
 F 1 "SW_SPDT" H 1650 1616 50  0000 C CNN
 F 2 "" H 1650 1850 50  0001 C CNN
@@
 	1350 1750 1350 1650
 $Comp
-L power:GND #PWR?
+L power:GND #PWR03
 U 1 1 6193FF44
 P 1350 2000
-F 0 "#PWR?" H 1350 1750 50  0001 C CNN
+F 0 "#PWR03" H 1350 1750 50  0001 C CNN
 F 1 "GND" H 1355 1827 50  0000 C CNN
 F 2 "" H 1350 2000 50  0001 C CNN
@@
 	1350 1950 1350 2000
 $Comp
-L Device:R_Small R?
+L Device:R_Small R1
 U 1 1 61940DE7
 P 2050 1850
-F 0 "R?" V 1854 1850 50  0000 C CNN
+F 0 "R1" V 1854 1850 50  0000 C CNN
 F 1 "10k" V 1945 1850 50  0000 C CNN
 F 2 "" H 2050 1850 50  0001 C CNN
@@
 $EndComp
 $Comp
-L Switch:SW_Push SW?
+L Switch:SW_Push SW2
 U 1 1 61942FCD
 P 2600 1150
-F 0 "SW?" H 2600 1435 50  0000 C CNN
+F 0 "SW2" H 2600 1435 50  0000 C CNN
 F 1 "SW_Push" H 2600 1344 50  0000 C CNN
 F 2 "" H 2600 1350 50  0001 C CNN
@@
 	1850 1850 1950 1850
 $Comp
-L power:GND #PWR?
+L power:GND #PWR05
 U 1 1 6194CE67
 P 2350 1500
-F 0 "#PWR?" H 2350 1250 50  0001 C CNN
+F 0 "#PWR05" H 2350 1250 50  0001 C CNN
 F 1 "GND" H 2355 1327 50  0000 C CNN
 F 2 "" H 2350 1500 50  0001 C CNN
@@
 	2150 1850 2950 1850
 $Comp
-L Device:C_Small C?
+L Device:C_Small C1
 U 1 1 619518C0
 P 2600 1400
-F 0 "C?" H 2692 1446 50  0000 L CNN
+F 0 "C1" H 2692 1446 50  0000 L CNN
 F 1 "100nF" H 2692 1355 50  0000 L CNN
 F 2 "" H 2600 1400 50  0001 C CNN
@@
 	2350 1400 2350 1500
 $Comp
-L Device:C_Small C?
+L Device:C_Small C4
 U 1 1 61960CDC
 P 8050 5600
-F 0 "C?" H 8142 5646 50  0000 L CNN
+F 0 "C4" H 8142 5646 50  0000 L CNN
 F 1 "4.7uF" H 8142 5555 50  0000 L CNN
 F 2 "" H 8050 5600 50  0001 C CNN
@@
 $EndComp
 $Comp
-L Device:C_Small C?
+L Device:C_Small C5
 U 1 1 61960F53
 P 8400 5600
-F 0 "C?" H 8492 5646 50  0000 L CNN
+F 0 "C5" H 8492 5646 50  0000 L CNN
 F 1 "100nF" H 8492 5555 50  0000 L CNN
 F 2 "" H 8400 5600 50  0001 C CNN
@@
 $EndComp
 $Comp
-L Device:C_Small C?
+L Device:C_Small C6
 U 1 1 61961266
 P 8750 5600
-F 0 "C?" H 8842 5646 50  0000 L CNN
+F 0 "C6" H 8842 5646 50  0000 L CNN
 F 1 "100nF" H 8842 5555 50  0000 L CNN
 F 2 "" H 8750 5600 50  0001 C CNN
@@
 $EndComp
 $Comp
-L Device:C_Small C?
+L Device:C_Small C7
 U 1 1 619614B2
 P 9100 5600
-F 0 "C?" H 9192 5646 50  0000 L CNN
+F 0 "C7" H 9192 5646 50  0000 L CNN
 F 1 "100nF" H 9192 5555 50  0000 L CNN
 F 2 "" H 9100 5600 50  0001 C CNN
@@
 $EndComp
 $Comp
-L Device:C_Small C?
+L Device:C_Small C8
 U 1 1 6196177D
 P 9450 5600
-F 0 "C?" H 9542 5646 50  0000 L CNN
+F 0 "C8" H 9542 5646 50  0000 L CNN
 F 1 "1uF" H 9542 5555 50  0000 L CNN
 F 2 "" H 9450 5600 50  0001 C CNN
@@
 $EndComp
 $Comp
-L Device:C_Small C?
+L Device:C_Small C9
 U 1 1 61961A31
 P 9800 5600
-F 0 "C?" H 9892 5646 50  0000 L CNN
+F 0 "C9" H 9892 5646 50  0000 L CNN
 F 1 "10nF" H 9892 5555 50  0000 L CNN
 F 2 "" H 9800 5600 50  0001 C CNN
@@
 $EndComp
 $Comp
-L Device:C_Small C?
+L Device:C_Small C10
 U 1 1 61961CB5
 P 10150 5600
-F 0 "C?" H 10242 5646 50  0000 L CNN
+F 0 "C10" H 10242 5646 50  0000 L CNN
 F 1 "4.7uF" H 10242 5555 50  0000 L CNN
 F 2 "" H 10150 5600 50  0001 C CNN
@@
 $EndComp
 $Comp
-L Device:C_Small C?
+L Device:C_Small C11
 U 1 1 61961E5C
 P 10500 5600
-F 0 "C?" H 10592 5646 50  0000 L CNN
+F 0 "C11" H 10592 5646 50  0000 L CNN
 F 1 "100nF" H 10592 5555 50  0000 L CNN
 F 2 "" H 10500 5600 50  0001 C CNN
@@
 $EndComp
 $Comp
-L power:+3.3V #PWR?
+L power:+3.3V #PWR013
 U 1 1 6196203D
 P 8050 5350
-F 0 "#PWR?" H 8050 5200 50  0001 C CNN
+F 0 "#PWR013" H 8050 5200 50  0001 C CNN
 F 1 "+3.3V" H 8065 5523 50  0000 C CNN
 F 2 "" H 8050 5350 50  0001 C CNN
@@
 	10150 5500 10500 5500
 $Comp
-L power:GND #PWR?
+L power:GND #PWR014
 U 1 1 61964DFD
 P 8050 5850
-F 0 "#PWR?" H 8050 5600 50  0001 C CNN
+F 0 "#PWR014" H 8050 5600 50  0001 C CNN
 F 1 "GND" H 8055 5677 50  0000 C CNN
 F 2 "" H 8050 5850 50  0001 C CNN

Commit message: Big changes
Parts:
- removed R3: 5.1k, Resistor_SMD:R_0805_2012Metric, symbol Device:R_Small
- added C12, C13, C14, C15, C16, C17, C18, C19: 1uF, Capacitor_SMD:C_0402_1005Metric, symbol Device:C_Small
- added C20, C21: 10nF, Capacitor_SMD:C_0402_1005Metric, symbol Device:C_Small
- added R1: 5.1k, Resistor_SMD:R_0402_1005Metric, symbol Device:R_Small
- added R6, R7, R8, R9: 10k, Resistor_SMD:R_0603_1608Metric, symbol Device:R_Small
- added SW3: Rotary_Encoder_Switch, Rotary_Encoder:RotaryEncoder_Alps_EC11E-Switch_Vertical_H20mm, symbol Device:Rotary_Encoder_Switch
- added U3: NHD-C12832A1Z, thpd-kb01-custom:NHD-C12832A1Z, symbol thpd-kb01-custom:NHD-C12832A1Z
- C1: renamed from C2; footprint (none) -> Capacitor_SMD:C_0402_1005Metric
- C10: renamed from C11; footprint (none) -> Capacitor_SMD:C_0402_1005Metric
- C11: renamed from C1; footprint (none) -> Capacitor_SMD:C_0402_1005Metric
- C2: renamed from C3; footprint (none) -> Capacitor_SMD:C_0402_1005Metric
- C3: renamed from C4; footprint (none) -> Capacitor_SMD:C_0402_1005Metric
- C4: renamed from C5; footprint (none) -> Capacitor_SMD:C_0402_1005Metric
- C5: renamed from C6; footprint (none) -> Capacitor_SMD:C_0402_1005Metric
- C6: renamed from C7; footprint (none) -> Capacitor_SMD:C_0402_1005Metric
- C7: renamed from C8; footprint (none) -> Capacitor_SMD:C_0402_1005Metric
- C8: renamed from C9; footprint (none) -> Capacitor_SMD:C_0402_1005Metric
- C9: renamed from C10; footprint (none) -> Capacitor_SMD:C_0402_1005Metric
- R2: footprint Resistor_SMD:R_0805_2012Metric -> Resistor_SMD:R_0402_1005Metric
- R3: renamed from R5; footprint (none) -> Resistor_SMD:R_0402_1005Metric
- R4: footprint (none) -> Resistor_SMD:R_0402_1005Metric
- R5: renamed from R1; footprint (none) -> Resistor_SMD:R_0603_1608Metric
- SW1: renamed from SW2; footprint (none) -> Button_Switch_SMD:SW_Push_SPST_NO_Alps_SKRK
- SW2: renamed from SW1; footprint (none) -> thpd-kb01-custom:SW_SPDT_K3-1296S-E1
- renumbered U3 to U1, U1 to U4
Connections:
- net +3V3: now also R6.2, R7.2, U3.12 (VDD), U3.A
- net GND: now also C14.2, C15.2, C16.2, C17.2, C18.2, C19.2, C20.1, C21.2, R1.2, SW3.C, U3.11 (VSS), U3.K
- net at J1.A5 (CC1): now also R1.1
- net LCD_CS: now reaches U4.13 (PA3)
- net LCD_CS: now also U3.17 (/CS1)
- net LCD_RST: now reaches U4.14 (PA4)
- net LCD_RST: now also U3.16 (/RES)
- net SPI1_SCK: now reaches U4.15 (PA5)
- net SPI1_SCK: now also U3.14 (SCL)
- net LCD_A0: now reaches U4.16 (PA6)
- net LCD_A0: now also U3.15 (A0)
- net SPI1_MOSI: now reaches U4.17 (PA7)
- net SPI1_MOSI: now also U3.13 (SI)
- net D_USB-: now reaches R3.2, U4.32 (PA11)
- net at R4.2: now also U2.4 (I/O2); no longer U4.33 (PA12)
- net D+ renamed D_USB+
- net D_USB+: now also U4.33 (PA12); no longer U2.3 (I/O2)
- net D-: no longer names the net of R3.1
- net D-: now also U2.6 (I/O1); no longer U2.1 (I/O1)
- net DCONN+ renamed D_USB_CONN+
- net D_USB_CONN+: now also U2.3 (I/O2); no longer U2.4 (I/O2)
- net DCONN- renamed D_USB_CONN-
- net D_USB_CONN-: now also U2.1 (I/O1); no longer U2.6 (I/O1)
- new net: C18.1, U3.1 (V0)
- new net: C19.1, U3.10 (VOUT)
- new net: C17.1, U3.2 (V1)
- new net: C16.1, U3.3 (V2)
- new net: C15.1, U3.4 (V3)
- new net: C14.1, U3.5 (V4)
- new net: C13.1, U3.6 (C2-)
- new net: C13.2, U3.7 (C2+)
- new net: C12.2, U3.8 (C1+)
- new net: C12.1, U3.9 (C1-)
- new net: R7.1, R9.2, SW3.A
- new net: R6.1, R8.1, SW3.B
- new net ROT_A: C21.1, R9.1
- new net ROT_B: C20.2, R8.2
- new net ROT_SW_COL: SW3.S1
- new net ROT_SW_ROW: SW3.S2
Other:
- moved on the sheet: C1, C10, C11, C2, C3, C4, C5, C6, C7, C8, C9, F1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
