File: thpd-kb01-keys.sch (KiCad schematic (older format))
At the start: 216 parts

Commit message: wip
Parts:
- removed D? (x8): D_Small, symbol Device:D_Small
- removed MX? (x8): MX-NoLED, symbol MX_Alps_Hybrid:MX-NoLED
- D1, D10, D100, D11, D12, D13, D14, D15, D16, D17, D18, D19, D2, D20, D21, D22, D23, D24, D25, D26, D27, D28, D29, D3, D30, D31, D32, D33, D34, D35, D36, D37, D38, D39, D4, D40, D41, D42, D43, D44, D45, D46, D47, D48, D49, D5, D50, D51, D52, D53, D54, D55, D56, D57, D58, D59, D6, D60, D61, D62, D63, D64, D65, D66, D67, D68, D69, D7, D70, D71, D72, D73, D74, D75, D76, D77, D78, D79, D8, D80, D81, D82, D83, D84, D85, D86, D87, D88, D89, D9, D90, D91, D92, D93, D94, D95, D96, D97, D98, D99: renamed from D?; footprint (none) -> Diode_SMD:D_SOD-123
- MX10: renamed from MX?; value MX-NoLED -> A
- MX100: renamed from MX?; value MX-NoLED -> NumEnter
- MX11: renamed from MX?; value MX-NoLED -> Z
- MX13: renamed from MX?; value MX-NoLED -> F2
- MX14: renamed from MX?; value MX-NoLED -> 2
- MX15: renamed from MX?; value MX-NoLED -> W
- MX16: renamed from MX?; value MX-NoLED -> S
- MX17: renamed from MX?; value MX-NoLED -> X
- MX19: renamed from MX?; value MX-NoLED -> F3
- MX2: renamed from MX?; value MX-NoLED -> ~`
- MX20: renamed from MX?; value MX-NoLED -> 3
- MX21: renamed from MX?; value MX-NoLED -> E
- MX22: renamed from MX?; value MX-NoLED -> D
- MX23: renamed from MX?; value MX-NoLED -> C
- MX24: renamed from MX?; value Esc -> F4
- MX25: renamed from MX?; value MX-NoLED -> 4
- MX26: renamed from MX?; value MX-NoLED -> R
- MX27: renamed from MX?; value MX-NoLED -> F
- MX28: renamed from MX?; value MX-NoLED -> V
- MX29: renamed from MX?; value MX-NoLED -> F5
- MX3: renamed from MX?; value MX-NoLED -> Tab
- MX30: renamed from MX?; value MX-NoLED -> 5
- MX31: renamed from MX?; value MX-NoLED -> T
- MX32: renamed from MX?; value MX-NoLED -> G
- MX33: renamed from MX?; value MX-NoLED -> B
- MX34: renamed from MX?; value MX-NoLED -> Spacebar
- MX35: renamed from MX?; value MX-NoLED -> F6
- MX36: renamed from MX?; value MX-NoLED -> 6
- MX37: renamed from MX?; value MX-NoLED -> Y
- MX38: renamed from MX?; value MX-NoLED -> H
- MX39: renamed from MX?; value MX-NoLED -> N
- MX4: renamed from MX?; value MX-NoLED -> Caps Lock
- MX40: renamed from MX?; value MX-NoLED -> F7
- MX41: renamed from MX?; value MX-NoLED -> 7
- MX42: renamed from MX?; value MX-NoLED -> U
- MX43: renamed from MX?; value MX-NoLED -> J
- MX44: renamed from MX?; value MX-NoLED -> M
- MX45: renamed from MX?; value Esc -> F8
- MX46: renamed from MX?; value MX-NoLED -> 8
- MX47: renamed from MX?; value MX-NoLED -> I
- MX48: renamed from MX?; value MX-NoLED -> K
- MX49: renamed from MX?; value MX-NoLED -> <
- MX5: renamed from MX?; value MX-NoLED -> Shift
- MX50: renamed from MX?; value MX-NoLED -> F9
- MX51: renamed from MX?; value MX-NoLED -> 9
- MX52: renamed from MX?; value MX-NoLED -> O
- MX53: renamed from MX?; value MX-NoLED -> L
- MX54: renamed from MX?; value MX-NoLED -> >
- MX55: renamed from MX?; value MX-NoLED -> RAlt
- MX56: renamed from MX?; value MX-NoLED -> F10
- MX57: renamed from MX?; value MX-NoLED -> 0
- MX58: renamed from MX?; value MX-NoLED -> P
- MX59: renamed from MX?; value MX-NoLED -> ;
- MX60: renamed from MX?; value MX-NoLED -> ?
- MX61: renamed from MX?; value MX-NoLED -> RFn
- MX62: renamed from MX?; value MX-NoLED -> F11
- MX63: renamed from MX?; value MX-NoLED -> -
- MX64: renamed from MX?; value MX-NoLED -> {
- MX65: renamed from MX?; value MX-NoLED -> '
- MX66: renamed from MX?; value MX-NoLED -> RShift
- MX67: renamed from MX?; value MX-NoLED -> RCtrl
- MX68: renamed from MX?; value Esc -> F12
- MX69: renamed from MX?; value MX-NoLED -> =
- MX7: renamed from MX?; value MX-NoLED -> F1
- MX70: renamed from MX?; value MX-NoLED -> }
- MX71: renamed from MX?; value MX-NoLED -> LeftArrow
- MX72: renamed from MX?; value MX-NoLED -> \\
- MX73: renamed from MX?; value MX-NoLED -> Backspace
- MX74: renamed from MX?; value MX-NoLED -> Enter
- MX75: renamed from MX?; value MX-NoLED -> UpArrow
- MX76: renamed from MX?; value MX-NoLED -> DownArrow
- MX77: renamed from MX?; value MX-NoLED -> PrtScr
- MX78: renamed from MX?; value MX-NoLED -> Home
- MX79: renamed from MX?; value MX-NoLED -> PageUp
- MX8: renamed from MX?; value MX-NoLED -> 1
- MX80: renamed from MX?; value MX-NoLED -> PageDown
- MX81: renamed from MX?; value MX-NoLED -> End
- MX82: renamed from MX?; value MX-NoLED -> RightArrow
- MX83: renamed from MX?; value MX-NoLED -> Delete
- MX84: renamed from MX?; value MX-NoLED -> NumLock
- MX85: renamed from MX?; value MX-NoLED -> Num7
- MX86: renamed from MX?; value MX-NoLED -> Num4
- MX87: renamed from MX?; value MX-NoLED -> Num1
- MX88: renamed from MX?; value MX-NoLED -> Num0
- MX89: renamed from MX?; value MX-NoLED -> Num-
- MX9: renamed from MX?; value MX-NoLED -> Q
- MX90: renamed from MX?; value MX-NoLED -> /
- MX91: renamed from MX?; value MX-NoLED -> Num8
- MX92: renamed from MX?; value MX-NoLED -> Num5
- MX93: renamed from MX?; value MX-NoLED -> Num2
- MX94: renamed from MX?; value MX-NoLED -> Num.
- MX95: renamed from MX?; value MX-NoLED -> Num+
- MX96: renamed from MX?; value MX-NoLED -> *
- MX97: renamed from MX?; value MX-NoLED -> Num9
- MX98: renamed from MX?; value MX-NoLED -> Num6
- MX99: renamed from MX?; value MX-NoLED -> Num3
- gave numbers to parts that had none: 4
Connections:
- net labels added: COL1, COL10, COL11, COL12, COL13, COL14, COL15, COL16, COL17, COL2, COL3, COL4, COL5, COL6, COL7, COL8, COL9
- wire segments 324 -> 300
Other:
- moved on the sheet: D1, D10, D100, D11, D12, D13, D14, D15, D16, D17, D18, D19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

Commit message: wip
Parts:
- MX1, MX10, MX11, MX13, MX14, MX15, MX16, MX17, MX19, MX2, MX20, MX21, MX22, MX23, MX24, MX25, MX26, MX27, MX28, MX29, MX30, MX31, MX32, MX33, MX35, MX36, MX37, MX38, MX39, MX40, MX41, MX42, MX43, MX44, MX45, MX46, MX47, MX48, MX49, MX50, MX51, MX52, MX53, MX54, MX55, MX56, MX57, MX58, MX59, MX60, MX61, MX62, MX63, MX64, MX65, MX67, MX68, MX69, MX7, MX70, MX71, MX72, MX75, MX76, MX77, MX78, MX79, MX8, MX80, MX81, MX82, MX83, MX84, MX85, MX86, MX87, MX89, MX9, MX90, MX91, MX92, MX93, MX94, MX96, MX97, MX98, MX99: footprint (none) -> MX_Alps_Hybrid:MX-1U-NoLED
- MX100, MX73, MX88, MX95: footprint (none) -> MX_Alps_Hybrid:MX-2U-NoLED
- MX12, MX18, MX6: footprint (none) -> MX_Alps_Hybrid:MX-1.25U-NoLED
- MX3: footprint (none) -> MX_Alps_Hybrid:MX-1.5U-NoLED
- MX34: footprint (none) -> MX_Alps_Hybrid:MX-6.25U-NoLED
- MX4, MX66: footprint (none) -> MX_Alps_Hybrid:MX-1.75U-NoLED
- MX5: footprint (none) -> MX_Alps_Hybrid:MX-2.25U-NoLED
- MX74: footprint (none) -> MX_Alps_Hybrid:MX-ISO

Commit message: wip pcb
Connections:
- net COL11: no longer MX66.1 (COL)
- net COL12: now also MX66.1 (COL)
Other:
- moved on the sheet: D66, MX66
Changed lines of the file:
@@
 L MX_Alps_Hybrid:MX-NoLED MX66
 U 1 1 618BED9D
-P 6650 4700
-F 0 "MX66" H 6683 4923 60  0000 C CNN
-F 1 "RShift" H 6683 4849 20  0000 C CNN
-F 2 "MX_Alps_Hybrid:MX-1.75U-NoLED" H 6025 4675 60  0001 C CNN
-F 3 "" H 6025 4675 60  0001 C CNN
-	1    6650 4700
+P 7100 4700
+F 0 "MX66" H 7133 4923 60  0000 C CNN
+F 1 "RShift" H 7133 4849 20  0000 C CNN
+F 2 "MX_Alps_Hybrid:MX-1.75U-NoLED" H 6475 4675 60  0001 C CNN
+F 3 "" H 6475 4675 60  0001 C CNN
+	1    7100 4700
 	1    0    0    -1
 $EndComp
@@
 L Device:D_Small D66
 U 1 1 618BEDA7
-P 6500 4950
-F 0 "D66" V 6546 4880 50  0000 R CNN
-F 1 "D_Small" V 6455 4880 50  0000 R CNN
-F 2 "Diode_SMD:D_SOD-123" V 6500 4950 50  0001 C CNN
-F 3 "~" V 6500 4950 50  0001 C CNN
-	1    6500 4950
-	0    -1   -1   0
-$EndComp
-Wire Wire Line
-	6500 4850 6600 4850
+P 6950 4950
+F 0 "D66" V 6996 4880 50  0000 R CNN
+F 1 "D_Small" V 6905 4880 50  0000 R CNN
+F 2 "Diode_SMD:D_SOD-123" V 6950 4950 50  0001 C CNN
+F 3 "~" V 6950 4950 50  0001 C CNN
+	1    6950 4950
+	0    -1   -1   0
+$EndComp
 $Comp
 L MX_Alps_Hybrid:MX-NoLED MX67
@@
 	5550 5050 6000 5050
 Connection ~ 6000 5050
-Wire Wire Line
-	6000 5050 6500 5050
-Connection ~ 6500 5050
 Connection ~ 7450 5050
 Wire Wire Line
@@
 Wire Wire Line
 	6300 4650 6300 4000
-Wire Wire Line
-	6800 5300 6800 4650
 Connection ~ 6800 2050
 Connection ~ 6800 2700
@@
 Wire Wire Line
 	6800 4000 6800 3350
-Connection ~ 6800 4650
-Wire Wire Line
-	6800 4650 6800 4000
 Connection ~ 7250 2050
 Connection ~ 7250 2700
@@
 	8400 5700 8850 5700
 Wire Wire Line
-	6500 5050 7450 5050
-Wire Wire Line
 	8200 3350 8200 4000
 Connection ~ 8400 2450
@@
 	6500 4400 7900 4400
 Wire Wire Line
-	7250 3350 7250 5300
+	7250 3350 7250 4650
 Connection ~ 8850 5700
 Wire Wire Line
@@
 Text HLabel 9600 1500 1    50   Input ~ 0
 COL17
+Connection ~ 7250 4650
+Wire Wire Line
+	7250 4650 7250 5300
+Wire Wire Line
+	6800 4000 6800 5300
+Connection ~ 6950 5050
+Wire Wire Line
+	6950 5050 7450 5050
+Wire Wire Line
+	6000 5050 6950 5050
+Wire Wire Line
+	6950 4850 7050 4850
 $EndSCHEMATC

Commit message: wip
Parts:
- D1, D10, D100, D11, D12, D13, D14, D15, D16, D17, D18, D19, D2, D20, D21, D22, D23, D24, D25, D26, D27, D28, D29, D3, D30, D31, D32, D33, D34, D35, D36, D37, D38, D39, D4, D40, D41, D42, D43, D44, D45, D46, D47, D48, D49, D5, D50, D51, D52, D53, D54, D55, D56, D57, D58, D59, D6, D60, D61, D62, D63, D64, D65, D66, D67, D68, D69, D7, D70, D71, D72, D73, D74, D75, D76, D77, D78, D79, D8, D80, D81, D82, D83, D84, D85, D86, D87, D88, D89, D9, D90, D91, D92, D93, D94, D95, D96, D97, D98, D99: footprint Diode_SMD:D_SOD-123 -> Diode_SMD:D_SOD-123F
- MX1, MX10, MX11, MX13, MX14, MX15, MX16, MX17, MX19, MX2, MX20, MX21, MX22, MX23, MX24, MX25, MX26, MX27, MX28, MX29, MX30, MX31, MX32, MX33, MX35, MX36, MX37, MX38, MX39, MX40, MX41, MX42, MX43, MX44, MX45, MX46, MX47, MX48, MX49, MX50, MX51, MX52, MX53, MX54, MX55, MX56, MX57, MX58, MX59, MX60, MX61, MX62, MX63, MX64, MX65, MX67, MX68, MX69, MX7, MX70, MX71, MX72, MX75, MX76, MX77, MX78, MX79, MX8, MX80, MX81, MX82, MX83, MX84, MX85, MX86, MX87, MX89, MX9, MX90, MX91, MX92, MX93, MX94, MX96, MX97, MX98, MX99: footprint MX_Alps_Hybrid:MX-1U-NoLED -> Button_Switch_Keyboard:SW_Cherry_MX_1.00u_Plate
- MX100, MX95: footprint MX_Alps_Hybrid:MX-2U-NoLED -> Button_Switch_Keyboard:SW_Cherry_MX_2.00u_Vertical_Plate
- MX12, MX18, MX6: footprint MX_Alps_Hybrid:MX-1.25U-NoLED -> Button_Switch_Keyboard:SW_Cherry_MX_1.25u_Plate
- MX3: footprint MX_Alps_Hybrid:MX-1.5U-NoLED -> Button_Switch_Keyboard:SW_Cherry_MX_1.50u_Plate
- MX34: footprint MX_Alps_Hybrid:MX-6.25U-NoLED -> Button_Switch_Keyboard:SW_Cherry_MX_6.25u_Plate
- MX4, MX66: footprint MX_Alps_Hybrid:MX-1.75U-NoLED -> Button_Switch_Keyboard:SW_Cherry_MX_1.75u_Plate
- MX5: footprint MX_Alps_Hybrid:MX-2.25U-NoLED -> Button_Switch_Keyboard:SW_Cherry_MX_2.25u_Plate
- MX73, MX88: footprint MX_Alps_Hybrid:MX-2U-NoLED -> Button_Switch_Keyboard:SW_Cherry_MX_2.00u_Plate
- MX74: footprint MX_Alps_Hybrid:MX-ISO -> Button_Switch_Keyboard:SW_Cherry_MX_ISOEnter_Plate

Commit message: re-annotate symbols
Parts:
- renumbered D67 to D66, D68 to D67, D69 to D68, D70 to D69, D66 to D70, MX67 to MX66, MX68 to MX67, MX69 to MX68, MX70 to MX69, MX66 to MX70
Changed lines of the file:
@@
 	6500 4200 6600 4200
 $Comp
-L MX_Alps_Hybrid:MX-NoLED MX66
+L MX_Alps_Hybrid:MX-NoLED MX70
 U 1 1 618BED9D
 P 7100 4700
-F 0 "MX66" H 7133 4923 60  0000 C CNN
+F 0 "MX70" H 7133 4923 60  0000 C CNN
 F 1 "RShift" H 7133 4849 20  0000 C CNN
 F 2 "Button_Switch_Keyboard:SW_Cherry_MX_1.75u_Plate" H 6475 4675 60  0001 C CNN
@@
 $EndComp
 $Comp
-L Device:D_Small D66
+L Device:D_Small D70
 U 1 1 618BEDA7
 P 6950 4950
-F 0 "D66" V 6996 4880 50  0000 R CNN
+F 0 "D70" V 6996 4880 50  0000 R CNN
 F 1 "D_Small" V 6905 4880 50  0000 R CNN
 F 2 "Diode_SMD:D_SOD-123F" V 6950 4950 50  0001 C CNN
@@
 $EndComp
 $Comp
-L MX_Alps_Hybrid:MX-NoLED MX67
+L MX_Alps_Hybrid:MX-NoLED MX66
 U 1 1 618BEDB2
 P 6650 5350
-F 0 "MX67" H 6683 5573 60  0000 C CNN
+F 0 "MX66" H 6683 5573 60  0000 C CNN
 F 1 "RCtrl" H 6683 5499 20  0000 C CNN
 F 2 "Button_Switch_Keyboard:SW_Cherry_MX_1.00u_Plate" H 6025 5325 60  0001 C CNN
@@
 $EndComp
 $Comp
-L Device:D_Small D67
+L Device:D_Small D66
 U 1 1 618BEDBC
 P 6500 5600
-F 0 "D67" V 6546 5530 50  0000 R CNN
+F 0 "D66" V 6546 5530 50  0000 R CNN
 F 1 "D_Small" V 6455 5530 50  0000 R CNN
 F 2 "Diode_SMD:D_SOD-123F" V 6500 5600 50  0001 C CNN
@@
 	6500 5500 6600 5500
 $Comp
-L MX_Alps_Hybrid:MX-NoLED MX68
+L MX_Alps_Hybrid:MX-NoLED MX67
 U 1 1 618BEDC7
 P 7100 2100
-F 0 "MX68" H 7133 2323 60  0000 C CNN
+F 0 "MX67" H 7133 2323 60  0000 C CNN
 F 1 "F12" H 7133 2249 20  0000 C CNN
 F 2 "Button_Switch_Keyboard:SW_Cherry_MX_1.00u_Plate" H 6475 2075 60  0001 C CNN
@@
 $EndComp
 $Comp
-L Device:D_Small D68
+L Device:D_Small D67
 U 1 1 618BEDD1
 P 6950 2350
-F 0 "D68" V 6996 2280 50  0000 R CNN
+F 0 "D67" V 6996 2280 50  0000 R CNN
 F 1 "D_Small" V 6905 2280 50  0000 R CNN
 F 2 "Diode_SMD:D_SOD-123F" V 6950 2350 50  0001 C CNN
@@
 	6950 2250 7050 2250
 $Comp
-L MX_Alps_Hybrid:MX-NoLED MX69
+L MX_Alps_Hybrid:MX-NoLED MX68
 U 1 1 618BEDDC
 P 7100 2750
-F 0 "MX69" H 7133 2973 60  0000 C CNN
+F 0 "MX68" H 7133 2973 60  0000 C CNN
 F 1 "=" H 7133 2899 20  0000 C CNN
 F 2 "Button_Switch_Keyboard:SW_Cherry_MX_1.00u_Plate" H 6475 2725 60  0001 C CNN
@@
 $EndComp
 $Comp
-L Device:D_Small D69
+L Device:D_Small D68
 U 1 1 618BEDE6
 P 6950 3000
-F 0 "D69" V 6996 2930 50  0000 R CNN
+F 0 "D68" V 6996 2930 50  0000 R CNN
 F 1 "D_Small" V 6905 2930 50  0000 R CNN
 F 2 "Diode_SMD:D_SOD-123F" V 6950 3000 50  0001 C CNN
@@
 	6950 2900 7050 2900
 $Comp
-L MX_Alps_Hybrid:MX-NoLED MX70
+L MX_Alps_Hybrid:MX-NoLED MX69
 U 1 1 618BEDF1
 P 7100 3400
-F 0 "MX70" H 7133 3623 60  0000 C CNN
+F 0 "MX69" H 7133 3623 60  0000 C CNN
 F 1 "}" H 7133 3549 20  0000 C CNN
 F 2 "Button_Switch_Keyboard:SW_Cherry_MX_1.00u_Plate" H 6475 3375 60  0001 C CNN
@@
 $EndComp
 $Comp
-L Device:D_Small D70
+L Device:D_Small D69
 U 1 1 618BEDFB
 P 6950 3650
-F 0 "D70" V 6996 3580 50  0000 R CNN
+F 0 "D69" V 6996 3580 50  0000 R CNN
 F 1 "D_Small" V 6905 3580 50  0000 R CNN
 F 2 "Diode_SMD:D_SOD-123F" V 6950 3650 50  0001 C CNN

Commit message: Big changes
Parts:
- added D15, D17: D_Small, Diode_SMD:D_SOD-123, symbol Device:D_Small
- added MX15: F14, Button_Switch_Keyboard:SW_Cherry_MX_1.00u_Plate, symbol MX_Alps_Hybrid:MX-NoLED
- D1, D87: footprint Diode_SMD:D_SOD-123F -> Diode_SMD:D_SOD-123
- D10: renamed from D50; footprint Diode_SMD:D_SOD-123F -> Diode_SMD:D_SOD-123
- D100: renamed from D82; footprint Diode_SMD:D_SOD-123F -> Diode_SMD:D_SOD-123
- D101: renamed from D88; footprint Diode_SMD:D_SOD-123F -> Diode_SMD:D_SOD-123
- D102: renamed from D94; footprint Diode_SMD:D_SOD-123F -> Diode_SMD:D_SOD-123
- D11: renamed from D56; footprint Diode_SMD:D_SOD-123F -> Diode_SMD:D_SOD-123
- D12: renamed from D62; footprint Diode_SMD:D_SOD-123F -> Diode_SMD:D_SOD-123
- D13: renamed from D67; footprint Diode_SMD:D_SOD-123F -> Diode_SMD:D_SOD-123
- D14: renamed from D77; footprint Diode_SMD:D_SOD-123F -> Diode_SMD:D_SOD-123
- D16: renamed from D83; footprint Diode_SMD:D_SOD-123F -> Diode_SMD:D_SOD-123
- D18: renamed from D2; footprint Diode_SMD:D_SOD-123F -> Diode_SMD:D_SOD-123
- D19: renamed from D8; footprint Diode_SMD:D_SOD-123F -> Diode_SMD:D_SOD-123
- D2: renamed from D7; footprint Diode_SMD:D_SOD-123F -> Diode_SMD:D_SOD-123
- D20: renamed from D14; footprint Diode_SMD:D_SOD-123F -> Diode_SMD:D_SOD-123
- D21: renamed from D20; footprint Diode_SMD:D_SOD-123F -> Diode_SMD:D_SOD-123
- D22: renamed from D25; footprint Diode_SMD:D_SOD-123F -> Diode_SMD:D_SOD-123
- D23: renamed from D30; footprint Diode_SMD:D_SOD-123F -> Diode_SMD:D_SOD-123
- D24: renamed from D36; footprint Diode_SMD:D_SOD-123F -> Diode_SMD:D_SOD-123
- D25: renamed from D41; footprint Diode_SMD:D_SOD-123F -> Diode_SMD:D_SOD-123
- D26: renamed from D46; footprint Diode_SMD:D_SOD-123F -> Diode_SMD:D_SOD-123
- D27: renamed from D51; footprint Diode_SMD:D_SOD-123F -> Diode_SMD:D_SOD-123
- D28: renamed from D57; footprint Diode_SMD:D_SOD-123F -> Diode_SMD:D_SOD-123
- D29: renamed from D63; footprint Diode_SMD:D_SOD-123F -> Diode_SMD:D_SOD-123
- D3: renamed from D13; footprint Diode_SMD:D_SOD-123F -> Diode_SMD:D_SOD-123
- D30: renamed from D68; footprint Diode_SMD:D_SOD-123F -> Diode_SMD:D_SOD-123
- D31: renamed from D73; footprint Diode_SMD:D_SOD-123F -> Diode_SMD:D_SOD-123
- D32: renamed from D78; footprint Diode_SMD:D_SOD-123F -> Diode_SMD:D_SOD-123
- D33: renamed from D84; footprint Diode_SMD:D_SOD-123F -> Diode_SMD:D_SOD-123
- D34: renamed from D90; footprint Diode_SMD:D_SOD-123F -> Diode_SMD:D_SOD-123
- D35: renamed from D96; footprint Diode_SMD:D_SOD-123F -> Diode_SMD:D_SOD-123
- D36: renamed from D89; footprint Diode_SMD:D_SOD-123F -> Diode_SMD:D_SOD-123
- D37: renamed from D3; footprint Diode_SMD:D_SOD-123F -> Diode_SMD:D_SOD-123
- D38: renamed from D9; footprint Diode_SMD:D_SOD-123F -> Diode_SMD:D_SOD-123
- D39: renamed from D15; footprint Diode_SMD:D_SOD-123F -> Diode_SMD:D_SOD-123
- D4: renamed from D19; footprint Diode_SMD:D_SOD-123F -> Diode_SMD:D_SOD-123
- D40: renamed from D21; footprint Diode_SMD:D_SOD-123F -> Diode_SMD:D_SOD-123
- D41: renamed from D26; footprint Diode_SMD:D_SOD-123F -> Diode_SMD:D_SOD-123
- D42: renamed from D31; footprint Diode_SMD:D_SOD-123F -> Diode_SMD:D_SOD-123
- D43: renamed from D37; footprint Diode_SMD:D_SOD-123F -> Diode_SMD:D_SOD-123
- D44: renamed from D42; footprint Diode_SMD:D_SOD-123F -> Diode_SMD:D_SOD-123
- D45: renamed from D47; footprint Diode_SMD:D_SOD-123F -> Diode_SMD:D_SOD-123
- D46: renamed from D52; footprint Diode_SMD:D_SOD-123F -> Diode_SMD:D_SOD-123
- D47: renamed from D58; footprint Diode_SMD:D_SOD-123F -> Diode_SMD:D_SOD-123
- D48: renamed from D64; footprint Diode_SMD:D_SOD-123F -> Diode_SMD:D_SOD-123
- D49: renamed from D69; footprint Diode_SMD:D_SOD-123F -> Diode_SMD:D_SOD-123
- D5: renamed from D24; footprint Diode_SMD:D_SOD-123F -> Diode_SMD:D_SOD-123
- D50: renamed from D74; footprint Diode_SMD:D_SOD-123F -> Diode_SMD:D_SOD-123
- D51: renamed from D79; footprint Diode_SMD:D_SOD-123F -> Diode_SMD:D_SOD-123
- D52: renamed from D85; footprint Diode_SMD:D_SOD-123F -> Diode_SMD:D_SOD-123
- D53: renamed from D91; footprint Diode_SMD:D_SOD-123F -> Diode_SMD:D_SOD-123
- D54: renamed from D97; footprint Diode_SMD:D_SOD-123F -> Diode_SMD:D_SOD-123
- D55: renamed from D95; footprint Diode_SMD:D_SOD-123F -> Diode_SMD:D_SOD-123
- D56: renamed from D4; footprint Diode_SMD:D_SOD-123F -> Diode_SMD:D_SOD-123
- D57: renamed from D10; footprint Diode_SMD:D_SOD-123F -> Diode_SMD:D_SOD-123
- D58: renamed from D16; footprint Diode_SMD:D_SOD-123F -> Diode_SMD:D_SOD-123
- D59: renamed from D22; footprint Diode_SMD:D_SOD-123F -> Diode_SMD:D_SOD-123
- D6: renamed from D29; footprint Diode_SMD:D_SOD-123F -> Diode_SMD:D_SOD-123
- D60: renamed from D27; footprint Diode_SMD:D_SOD-123F -> Diode_SMD:D_SOD-123
- D61: renamed from D32; footprint Diode_SMD:D_SOD-123F -> Diode_SMD:D_SOD-123
- D62: renamed from D38; footprint Diode_SMD:D_SOD-123F -> Diode_SMD:D_SOD-123
- D63: renamed from D43; footprint Diode_SMD:D_SOD-123F -> Diode_SMD:D_SOD-123
- D64: renamed from D48; footprint Diode_SMD:D_SOD-123F -> Diode_SMD:D_SOD-123
- D65: renamed from D53; footprint Diode_SMD:D_SOD-123F -> Diode_SMD:D_SOD-123
- D66: renamed from D59; footprint Diode_SMD:D_SOD-123F -> Diode_SMD:D_SOD-123
- D67: renamed from D65; footprint Diode_SMD:D_SOD-123F -> Diode_SMD:D_SOD-123
- D68: renamed from D72; footprint Diode_SMD:D_SOD-123F -> Diode_SMD:D_SOD-123
- D69: renamed from D80; footprint Diode_SMD:D_SOD-123F -> Diode_SMD:D_SOD-123
- D7: renamed from D35; footprint Diode_SMD:D_SOD-123F -> Diode_SMD:D_SOD-123
- D70: renamed from D86; footprint Diode_SMD:D_SOD-123F -> Diode_SMD:D_SOD-123
- D71: renamed from D92; footprint Diode_SMD:D_SOD-123F -> Diode_SMD:D_SOD-123
- D72: renamed from D98; footprint Diode_SMD:D_SOD-123F -> Diode_SMD:D_SOD-123
- D73: renamed from D5; footprint Diode_SMD:D_SOD-123F -> Diode_SMD:D_SOD-123
- D74: renamed from D11; footprint Diode_SMD:D_SOD-123F -> Diode_SMD:D_SOD-123
- D75: renamed from D17; footprint Diode_SMD:D_SOD-123F -> Diode_SMD:D_SOD-123
- D76: renamed from D23; footprint Diode_SMD:D_SOD-123F -> Diode_SMD:D_SOD-123
- D77: renamed from D28; footprint Diode_SMD:D_SOD-123F -> Diode_SMD:D_SOD-123
- D78: renamed from D33; footprint Diode_SMD:D_SOD-123F -> Diode_SMD:D_SOD-123
- D79: renamed from D39; footprint Diode_SMD:D_SOD-123F -> Diode_SMD:D_SOD-123
- D8: renamed from D40; footprint Diode_SMD:D_SOD-123F -> Diode_SMD:D_SOD-123
- D80: renamed from D44; footprint Diode_SMD:D_SOD-123F -> Diode_SMD:D_SOD-123
- D81: renamed from D49; footprint Diode_SMD:D_SOD-123F -> Diode_SMD:D_SOD-123
- D82: renamed from D54; footprint Diode_SMD:D_SOD-123F -> Diode_SMD:D_SOD-123
- D83: renamed from D60; footprint Diode_SMD:D_SOD-123F -> Diode_SMD:D_SOD-123
- D84: renamed from D70; footprint Diode_SMD:D_SOD-123F -> Diode_SMD:D_SOD-123
- D85: renamed from D75; footprint Diode_SMD:D_SOD-123F -> Diode_SMD:D_SOD-123
- D86: renamed from D81; footprint Diode_SMD:D_SOD-123F -> Diode_SMD:D_SOD-123
- D88: renamed from D93; footprint Diode_SMD:D_SOD-123F -> Diode_SMD:D_SOD-123
- D89: renamed from D99; footprint Diode_SMD:D_SOD-123F -> Diode_SMD:D_SOD-123
- D9: renamed from D45; footprint Diode_SMD:D_SOD-123F -> Diode_SMD:D_SOD-123
- D90: renamed from D100; footprint Diode_SMD:D_SOD-123F -> Diode_SMD:D_SOD-123
- D91: renamed from D6; footprint Diode_SMD:D_SOD-123F -> Diode_SMD:D_SOD-123
- D92: renamed from D12; footprint Diode_SMD:D_SOD-123F -> Diode_SMD:D_SOD-123
- D93: renamed from D18; footprint Diode_SMD:D_SOD-123F -> Diode_SMD:D_SOD-123
- D94: renamed from D34; footprint Diode_SMD:D_SOD-123F -> Diode_SMD:D_SOD-123
- D95: renamed from D55; footprint Diode_SMD:D_SOD-123F -> Diode_SMD:D_SOD-123
- D96: renamed from D61; footprint Diode_SMD:D_SOD-123F -> Diode_SMD:D_SOD-123
- D97: renamed from D66; footprint Diode_SMD:D_SOD-123F -> Diode_SMD:D_SOD-123
- D98: renamed from D71; footprint Diode_SMD:D_SOD-123F -> Diode_SMD:D_SOD-123
- D99: renamed from D76; footprint Diode_SMD:D_SOD-123F -> Diode_SMD:D_SOD-123
- MX14: renamed from MX77; value PrtScr -> F13
- MX17: renamed from MX2; value ~` -> Tilde/Backtick
- MX28: renamed from MX63; value - -> Hyphen
- MX29: renamed from MX68; value = -> Equals
- MX33: renamed from MX90; value / -> Num/
- MX34: renamed from MX96; value * -> Num*
- MX66: renamed from MX65; value ' -> SingleQuote
- renumbered MX50 to MX10, MX88 to MX100, MX94 to MX101, MX56 to MX11, MX62 to MX12, MX67 to MX13, MX83 to MX16, MX8 to MX18, MX14 to MX19, MX7 to MX2, MX25 to MX21, MX30 to MX22, MX36 to MX23, MX41 to MX24, MX46 to MX25, MX51 to MX26, MX57 to MX27, MX13 to MX3, MX73 to MX30, MX78 to MX31, MX84 to MX32, MX89 to MX35, MX3 to MX36, MX9 to MX37, MX15 to MX38, MX21 to MX39, MX19 to MX4, MX26 to MX40, MX31 to MX41, MX37 to MX42, MX42 to MX43, MX47 to MX44, MX52 to MX45, MX58 to MX46, MX64 to MX47, MX69 to MX48, MX74 to MX49, MX24 to MX5, MX79 to MX50, MX85 to MX51, MX91 to MX52, MX97 to MX53, MX95 to MX54, MX4 to MX55, MX10 to MX56, MX16 to MX57, MX22 to MX58, MX27 to MX59, MX29 to MX6, MX32 to MX60, MX38 to MX61, MX43 to MX62, MX48 to MX63, MX53 to MX64, MX59 to MX65, MX72 to MX67, MX80 to MX68, MX86 to MX69, MX35 to MX7, MX92 to MX70, MX98 to MX71, MX5 to MX72, MX11 to MX73, MX17 to MX74, MX23 to MX75, MX28 to MX76, MX33 to MX77, MX39 to MX78, MX44 to MX79, MX40 to MX8, MX49 to MX80, MX54 to MX81, MX60 to MX82, MX70 to MX83, MX75 to MX84, MX81 to MX85, MX87 to MX86, MX93 to MX87, MX99 to MX88, MX100 to MX89, MX45 to MX9, MX6 to MX90, MX12 to MX91, MX18 to MX92, MX34 to MX93, MX55 to MX94, MX61 to MX95, MX66 to MX96, MX71 to MX97, MX76 to MX98, MX82 to MX99
Connections:
- net COL12: now also MX67.1 (COL)
- net COL13: now also MX14.1 (COL); no longer MX67.1 (COL)
- net COL14: now also MX15.1 (COL); no longer MX14.1 (COL)
- net COL16: no longer MX101.1 (COL), MX35.1 (COL)
- net COL17: now also MX101.1 (COL); no longer MX54.1 (COL), MX89.1 (COL)
- net ROW0: now also D15.1 (K), D17.1 (K); no longer D36.1 (K), D55.1 (K), D68.1 (K)
- net ROW1: now also D36.1 (K)
- net ROW2: now also D55.1 (K)
- net ROW3: now also D68.1 (K)
- net ROW4: now also D90.1 (K)
- net ROW5: no longer D90.1 (K)
- new net: D15.2 (A), MX15.2 (ROW)
- new net ROT_SW_COL: MX35.1 (COL), MX54.1 (COL), MX89.1 (COL)
- new net ROT_SW_ROW: D17.2 (A)
Other:
- moved on the sheet: D102, D14, D36, D55, D68, D90, MX101, MX14, MX35, MX54, MX67, MX89

Commit message: WIP
Parts:
- renumbered D101 to D100, D102 to D101, D17 to D102, D18 to D17, D19 to D18, D20 to D19, D21 to D20, D22 to D21, D23 to D22, D24 to D23, D25 to D24, D26 to D25, D27 to D26, D28 to D27, D29 to D28, D30 to D29, D31 to D30, D32 to D31, D33 to D32, D34 to D33, D35 to D34, D36 to D35, D37 to D36, D38 to D37, D39 to D38, D40 to D39, D41 to D40, D42 to D41, D43 to D42, D44 to D43, D45 to D44, D46 to D45, D47 to D46, D48 to D47, D49 to D48, D50 to D49, D51 to D50, D52 to D51, D53 to D52, D54 to D53, D55 to D54, D56 to D55, D57 to D56, D58 to D57, D59 to D58, D60 to D59, D61 to D60, D62 to D61, D63 to D62, D64 to D63, D65 to D64, D66 to D65, D67 to D66, D68 to D67, D69 to D68, D70 to D69, D71 to D70, D72 to D71, D73 to D72, D74 to D73, D75 to D74, D76 to D75, D77 to D76, D78 to D77, D79 to D78, D80 to D79, D81 to D80, D82 to D81, D83 to D82, D84 to D83, D85 to D84, D86 to D85, D87 to D86, D88 to D87, D89 to D88, D90 to D89, D91 to D90, D92 to D91, D93 to D92, D94 to D93, D95 to D94, D96 to D95, D97 to D96, D98 to D97, D99 to D98, D100 to D99

Commit message: Add LCSC part numbers and prepared for output.
Parts:
- D1, D10, D100, D101, D102, D11, D12, D13, D14, D15, D16, D17, D18, D19, D2, D20, D21, D22, D23, D24, D25, D26, D27, D28, D29, D3, D30, D31, D32, D33, D34, D35, D36, D37, D38, D39, D4, D40, D41, D42, D43, D44, D45, D46, D47, D48, D49, D5, D50, D51, D52, D53, D54, D55, D56, D57, D58, D59, D6, D60, D61, D62, D63, D64, D65, D66, D67, D68, D69, D7, D70, D71, D72, D73, D74, D75, D76, D77, D78, D79, D8, D80, D81, D82, D83, D84, D85, D86, D87, D88, D89, D9, D90, D91, D92, D93, D94, D95, D96, D97, D98, D99: LCSC Part # (none) -> C81598
